File: kicad/pong/pong.kicad_pcb (KiCad board)
At the start: 2 copper layers, 0 parts

Commit message: Add an interactive board view for Pong
Builds the board layout from assembly drawing A001433 Rev E — all 66 ICs at
their silkscreened A-H x 1-9 grid positions plus 34 discretes — and generates
an InteractiveHtmlBom view, embedded on the board page. Clicking a BOM row
finds the part on the board and vice versa.

The +5V and GND rails are wired and verified against each device's datasheet,
including the three that break the usual TTL convention: 7490/7493 take power
on 5/10, 7483 on 5/12, and the 555s on 8/1. Signal nets still need tracing
from schematic 002826, so net highlighting covers the rails only.

pcbnew quirks worth knowing (recorded in AGENTS.md):
- board.Remove() corrupts SWIG's type registry for the rest of the process;
  every later FootprintLoad() returns a bare pointer. Build a fresh board.
- PCB_IO_MGR.FindPlugin() hands back a manager-owned object that gets freed
  mid-run; construct PCB_IO_KICAD_SEXPR() instead.
- IBOM omits nets unless --include-nets is passed, which looks identical to
  having no netlist at all.

Co-Authored-By: Claude Opus 5 <noreply@anthropic.com>
Parts:
- added C1: 8000uF, CP_Radial_D16.0mm_P7.50mm, F.Cu at (238.0, 62.0)
- added C10: 0.1uF, C_Disc_D5.0mm_W2.5mm_P5.00mm, F.Cu at (203.8, 9.00)
- added C11: 0.1uF, C_Disc_D5.0mm_W2.5mm_P5.00mm, F.Cu at (229.2, 9.00)
- added C12: 1.0uF, C_Disc_D7.5mm_W2.5mm_P5.00mm, F.Cu at (120.0, 158.0)
- added C13: 5.0uF, CP_Radial_D5.0mm_P2.50mm, F.Cu at (134.0, 158.0)
- added C2: 470uF, CP_Radial_D10.0mm_P5.00mm, F.Cu at (238.0, 82.0)
- added C3: 0.1uF, C_Disc_D5.0mm_W2.5mm_P5.00mm, F.Cu at (26.0, 9.00)
- added C4: 0.1uF, C_Disc_D5.0mm_W2.5mm_P5.00mm, F.Cu at (51.4, 9.00)
- added C5: 0.1uF, C_Disc_D5.0mm_W2.5mm_P5.00mm, F.Cu at (76.8, 9.00)
- added C6: 0.1uF, C_Disc_D5.0mm_W2.5mm_P5.00mm, F.Cu at (102.2, 9.00)
- added C7: 0.1uF, C_Disc_D5.0mm_W2.5mm_P5.00mm, F.Cu at (127.6, 9.00)
- added C8: 0.1uF, C_Disc_D5.0mm_W2.5mm_P5.00mm, F.Cu at (153.0, 9.00)
- added C9: 0.1uF, C_Disc_D5.0mm_W2.5mm_P5.00mm, F.Cu at (178.4, 9.00)
- added D1: 1N4001, D_DO-41_SOD81_P10.16mm_Horizontal, F.Cu at (238.0, 96.0)
- added D2: 1N4001, D_DO-41_SOD81_P10.16mm_Horizontal, F.Cu at (238.0, 104.0)
- added D3: 1N4001, D_DO-41_SOD81_P10.16mm_Horizontal, F.Cu at (238.0, 112.0)
- added D4: 1N4001, D_DO-41_SOD81_P10.16mm_Horizontal, F.Cu at (238.0, 120.0)
- added D5: 1N914, D_DO-35_SOD27_P7.62mm_Horizontal, F.Cu at (238.0, 128.0)
- added J1: Edge Connector, PinHeader_1x15_P2.54mm_Vertical, F.Cu at (8.00, 60.0)
- added Q1: 2N3643, TO-92-2, F.Cu at (226.0, 140.0)
- added Q2: 2N3644, TO-92-2, F.Cu at (232.0, 140.0)
- added R1: 2.2M, R_Axial_DIN0207_L6.3mm_D2.5mm_P10.16mm_Horizontal, F.Cu at (214.0, 24.0)
- added R10: 50K, R_Axial_DIN0207_L6.3mm_D2.5mm_P10.16mm_Horizontal, F.Cu at (214.0, 78.0)
- added R2: 330K, R_Axial_DIN0207_L6.3mm_D2.5mm_P10.16mm_Horizontal, F.Cu at (214.0, 30.0)
- added R3: 2.2K, R_Axial_DIN0207_L6.3mm_D2.5mm_P10.16mm_Horizontal, F.Cu at (214.0, 36.0)
- added R4: 1K, R_Axial_DIN0207_L6.3mm_D2.5mm_P10.16mm_Horizontal, F.Cu at (214.0, 42.0)
- added R5: 1M, R_Axial_DIN0207_L6.3mm_D2.5mm_P10.16mm_Horizontal, F.Cu at (214.0, 48.0)
- added R6: 330R, R_Axial_DIN0207_L6.3mm_D2.5mm_P10.16mm_Horizontal, F.Cu at (214.0, 54.0)
- added R7: 330R, R_Axial_DIN0207_L6.3mm_D2.5mm_P10.16mm_Horizontal, F.Cu at (214.0, 60.0)
- added R8: 100R, R_Axial_DIN0207_L6.3mm_D2.5mm_P10.16mm_Horizontal, F.Cu at (214.0, 66.0)
- added R9: 5.6K, R_Axial_DIN0207_L6.3mm_D2.5mm_P10.16mm_Horizontal, F.Cu at (214.0, 72.0)
- added RV1: 50K POT (Player 1), Potentiometer_Alpha_RD901F-40-00D_Single_Vertical, F.Cu at (210.0, 150.0)
- added RV2: 50K POT (Player 2), Potentiometer_Alpha_RD901F-40-00D_Single_Vertical, F.Cu at (228.0, 150.0)
- added UA2: 74107, DIP-14_W7.62mm, F.Cu at (51.4, 153.3)
- added UA3: 9316, DIP-16_W7.62mm, F.Cu at (76.8, 153.3)
- added UA4: 7486, DIP-14_W7.62mm, F.Cu at (102.2, 153.3)
- added UA5: 7474, DIP-14_W7.62mm, F.Cu at (127.6, 153.3)
- added UA6: 7450, DIP-14_W7.62mm, F.Cu at (153.0, 153.3)
- added UA7: 7420, DIP-14_W7.62mm, F.Cu at (178.4, 153.3)
- added UA8: 7493, DIP-14_W7.62mm, F.Cu at (203.8, 153.3)
- added UA9: 555, DIP-8_W7.62mm, F.Cu at (229.2, 153.3)
- added UB2: 7400, DIP-14_W7.62mm, F.Cu at (51.4, 134.3)
- added UB3: 9316, DIP-16_W7.62mm, F.Cu at (76.8, 134.3)
- added UB4: 7483, DIP-16_W7.62mm, F.Cu at (102.2, 134.3)
- added UB5: 7474, DIP-14_W7.62mm, F.Cu at (127.6, 134.3)
- added UB6: 7450, DIP-14_W7.62mm, F.Cu at (153.0, 134.3)
- added UB7: 7400, DIP-14_W7.62mm, F.Cu at (178.4, 134.3)
- added UB8: 7493, DIP-14_W7.62mm, F.Cu at (203.8, 134.3)
- added UB9: 555, DIP-8_W7.62mm, F.Cu at (229.2, 134.3)
- added UC1: 7400, DIP-14_W7.62mm, F.Cu at (26.0, 115.2)
- added UC2: 7474, DIP-14_W7.62mm, F.Cu at (51.4, 115.2)
- added UC3: 7400, DIP-14_W7.62mm, F.Cu at (76.8, 115.2)
- added UC4: 7410, DIP-14_W7.62mm, F.Cu at (102.2, 115.2)
- added UC5: 7448, DIP-16_W7.62mm, F.Cu at (127.6, 115.2)
- added UC6: 74153, DIP-16_W7.62mm, F.Cu at (153.0, 115.2)
- added UC7: 7490, DIP-14_W7.62mm, F.Cu at (178.4, 115.2)
- added UC8: 74107, DIP-14_W7.62mm, F.Cu at (203.8, 115.2)
- added UC9: 7404, DIP-14_W7.62mm, F.Cu at (229.2, 115.2)
- added UD1: 7404, DIP-14_W7.62mm, F.Cu at (26.0, 96.2)
- added UD2: 7402, DIP-14_W7.62mm, F.Cu at (51.4, 96.2)
- added UD3: 7430, DIP-14_W7.62mm, F.Cu at (76.8, 96.2)
- added UD4: 7410, DIP-14_W7.62mm, F.Cu at (102.2, 96.2)
- added UD5: 7410, DIP-14_W7.62mm, F.Cu at (127.6, 96.2)
- added UD6: 74153, DIP-16_W7.62mm, F.Cu at (153.0, 96.2)
- added UD7: 7490, DIP-14_W7.62mm, F.Cu at (178.4, 96.2)
- added UD8: 7410, DIP-14_W7.62mm, F.Cu at (203.8, 96.2)
- added UD9: 74107, DIP-14_W7.62mm, F.Cu at (229.2, 96.2)
- added UE1: 7400, DIP-14_W7.62mm, F.Cu at (26.0, 77.2)
- added UE2: 7410, DIP-14_W7.62mm, F.Cu at (51.4, 77.2)
- added UE3: 7427, DIP-14_W7.62mm, F.Cu at (76.8, 77.2)
- added UE4: 7404, DIP-14_W7.62mm, F.Cu at (102.2, 77.2)
- added UE5: 7427, DIP-14_W7.62mm, F.Cu at (127.6, 77.2)
- added UE6: 7400, DIP-14_W7.62mm, F.Cu at (153.0, 77.2)
- added UE7: 7474, DIP-14_W7.62mm, F.Cu at (178.4, 77.2)
- added UE8: 7493, DIP-14_W7.62mm, F.Cu at (203.8, 77.2)
- added UE9: 7493, DIP-14_W7.62mm, F.Cu at (229.2, 77.2)
- added UF1: 7433, DIP-14_W7.62mm, F.Cu at (26.0, 58.1)
- added UF2: 7425, DIP-14_W7.62mm, F.Cu at (51.4, 58.1)
- added UF3: 74107, DIP-14_W7.62mm, F.Cu at (76.8, 58.1)
- added UF4: 555, DIP-8_W7.62mm, F.Cu at (102.2, 58.1)
- added UF5: 7402, DIP-14_W7.62mm, F.Cu at (127.6, 58.1)
- added UF6: 74107, DIP-14_W7.62mm, F.Cu at (153.0, 58.1)
- added UF7: 7430, DIP-14_W7.62mm, F.Cu at (178.4, 58.1)
- added UF8: 7493, DIP-14_W7.62mm, F.Cu at (203.8, 58.1)
- added UF9: 7493, DIP-14_W7.62mm, F.Cu at (229.2, 58.1)
- added UG1: 7402, DIP-14_W7.62mm, F.Cu at (26.0, 39.0)
- added UG2: 7427, DIP-14_W7.62mm, F.Cu at (51.4, 39.0)
- added UG3: 7400, DIP-14_W7.62mm, F.Cu at (76.8, 39.0)
- added UG4: 555, DIP-8_W7.62mm, F.Cu at (102.2, 39.0)
- added UG5: 7410, DIP-14_W7.62mm, F.Cu at (127.6, 39.0)
- added UG6: 74107, DIP-14_W7.62mm, F.Cu at (153.0, 39.0)
- added UG7: 9316, DIP-16_W7.62mm, F.Cu at (178.4, 39.0)
- added UH1: 7400, DIP-14_W7.62mm, F.Cu at (26.0, 20.0)
- added UH2: 74107, DIP-14_W7.62mm, F.Cu at (51.4, 20.0)
- added UH3: 7474, DIP-14_W7.62mm, F.Cu at (76.8, 20.0)
- added UH4: 7400, DIP-14_W7.62mm, F.Cu at (102.2, 20.0)
- added UH5: 7400, DIP-14_W7.62mm, F.Cu at (127.6, 20.0)
- added UH6: 7420, DIP-14_W7.62mm, F.Cu at (153.0, 20.0)
- added UH7: 9316, DIP-16_W7.62mm, F.Cu at (178.4, 20.0)
- added VR1: LM309K, TO-3, F.Cu at (238.0, 28.0)
Other:
- board outline added: 247 x 165 mm
- rule pad_to_mask_clearance: 0.05 -> 0
