File: kicad/football/football.kicad_pcb (KiCad board)
At the start: 2 copper layers, 290 x 275 mm, 77 parts

Commit message: Publish the single-printing boards, with the caveat on the page
Nine machines had exactly one printing carrying an IC parts list, so the
two-printing rule excluded them. They are in now, flagged: Monte Carlo
79 devices, Outlaw 47, Sky Diver 38, Orbit 37, Indy 4 30, Triple Hunt
29, Super Breakout 18, Soccer 17, Starship 1 10. Twenty-five boards and
1,365 devices on the site.

The flag is not a footnote. singleSource puts a warning at the top of the
board page saying the board was read once and not cross-checked, that
every other board here required two independent sources to agree, and
that the reader should treat it as a lead and check the chip against the
board. The boards list carries a badge, and the chip lookup still names
the source on every row.

With no second printing to disagree with, the well-formedness guard is
the only check left, so two fixes to what it has to work with.

OCR destroys the logic family the same two ways every time: L read as 1,
S read as 8 or 5. 74LS08 comes back as 741808, 74LS74 as 74L874, 74S04
as 74504. repair_family undoes it by trying every split of the string
into family and function number and taking the repair only when exactly
one of them names a device the packaging table knows. Ambiguous, and the
device does not go on the map. Orbit went from 16 devices to 37 on this
alone, Super Breakout from 12 to 18, Starship 1 from 6 to 10.

And the count layout states its device twice as well — 'Integrated
Circuit, 74S74 L7' — which only the paren layout was using. That is what
finally named the device both Football printings spelled 74874: the 3rd
printing's description had it right all along. Football gains L7.

Fifteen more parts join the packaging table, KiCAD-verified where KiCAD
has them: 7476, 7495, 7496, 74156, 74241, 74279, 7489, NE556, LM723, and
Fairchild's 9300, 9301, 9322, 9334 — the numbering a mid-70s Atari board
uses before 74-series became the house standard.

Co-Authored-By: Claude Opus 5 <noreply@anthropic.com>
Parts:
- added UL7: 74S74, DIP-14_W7.62mm, F.Cu at (178.4, 75.2)

Commit message: Test whether manual prose gives functional blocks, on Football
It does, on some manuals, and the test was worth running because the
first hypothesis was wrong. The section names on the hand-read boards do
not come from manual prose at all — they are titles printed on the
drawing sheets. Asteroids' technical manual has thirty-five headings and
not one is a theory-of-operation block.

But some manuals do carry a theory chapter that names blocks with their
positions, and Football's is one. It gives the MPU at C2, gated address
buffers at B1 and C1, data buffers at E2, program ROM at P1, N1 and M1,
working RAM at M2 and N2, address decoding at B3, E3 and C7, and a
watchdog reset counter at A4.

What makes it trustworthy is that where it overlaps the parts-list
harvest, the two agree on function without having any source in common:
B1, C1 and E2 are 74LS244 buffers, and B3 and E3 are 7442 decoders. Five
blocks are applied to devices already on the map.

Three program ROMs are added at M1, N1 and P1, where the theory chapter
and MAME's dumps of real boards agree on position. 2K each, so the
2316/2716 class that socket entries confirm as 24-pin everywhere else in
this corpus. Football goes 78 to 81.

Eight more positions are logged and not drawn. C2, M2, N2, C7 and A4 are
named by the prose but prose gives a function and a location, never a
part number. N7, C5 and D5 are graphics memory MAME dumps, but MAME is
one source and this manual predates the socket entries that settle pin
counts, so their package is not established.

The honest yield: prose reaches ten to fifteen positions on a board of
eighty, and only on manuals that have a theory chapter. It is not a
route to sections for every board, and the false-positive rate on a
naive search is high — capacitor designators, connector numbers and TV
screen zones all look like grid cells.

Co-Authored-By: Claude Opus 5 <noreply@anthropic.com>
Parts:
- added UM1: 033026-02, DIP-24_W15.24mm, F.Cu at (26.0, 56.1)
- added UN1: 033027-02, DIP-24_W15.24mm, F.Cu at (26.0, 37.0)
- added UP1: 033028-01, DIP-24_W15.24mm, F.Cu at (26.0, 18.0)
