File: kicad/centipede/centipede.kicad_pcb (KiCad board)
At the start: 2 copper layers, 300 x 300 mm, 93 parts

Commit message: Place the memory devices the IC parts lists cannot reach
Atari stocks ROM, RAM and the microprocessor under its own part numbers
— 90-7033, 036175-01, 90-6013 — not as 37-series IC stock, so the IC
harvest cannot see them however well it reads. That is why Centipede's
ROMs were missing and Red Baron's map had ten devices. merge_memory.py
reads those rows from the same typeset parts lists, under the same rules
as the IC merge: the drawing wins where it exists, two documents must
agree, and nothing is placed whose package cannot be established.

Red Baron 10 to 15, Asteroids Deluxe 92 to 100, Tempest 83 to 88,
Centipede 93 to 95, Missile Command 83 to 85, Lunar Lander 60 to 62.
1,494 devices across the boards, all sized, none contradicted.

Establishing the packages took two corrections, and both were the same
mistake in different clothes.

The first attempt sized Atari stock numbers by correlating a part
against the contact count of the socket at the positions it occupies,
pooled across a machine's documents. That is not a near miss: it put the
2114 at 40 pins, on twelve positions of apparent evidence, because two
printings number the board differently and the correlation was reading
one printing's parts list against another's sockets. Confined to within
a single document it behaves — 33 stock numbers established, 90-6013 by
39 documents agreeing, and 90-7033 correctly refusing to answer rather
than answering wrongly. Those 33 are in packages.py with their
provenance.

The second was the same shape. MAME's dump size was sizing a part from
whatever MAME dumped at that cell, which on Red Baron meant sizing
036175-01 from a dump of 037000-01 — sizing the socket, not the chip.
MAME now sizes a part only when the dump is of that part. Red Baron
loses two devices and keeps thirteen that are right.

Four more parts are sized from MAME's dump sizes alone, where every set
carrying the part agrees and the era leaves no room: 32 bytes and 256
bytes are both bipolar PROMs in a 1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
Parts:
- added UA6: 137170-001, DIP-24_W15.24mm, F.Cu at (153.0, 265.6)
- added UB6: 137170-001, DIP-24_W15.24mm, F.Cu at (153.0, 246.6)
