File: kicad/fast-freddie/fast-freddie.kicad_pcb (KiCad board)
At the start: 2 copper layers, 300 x 300 mm, 93 parts

Commit message: Fill four thin boards and add four more, from the parts lists
The parts-list harvest was described as swept. It was swept for finding new
machines to hand-read; it had not been run against the boards already here.
Running it over all 2,389 cached documents finds 29 boards where there was
one, and 1,864 devices where there were 1,365.

Red Baron goes from 15 devices to 66 and Warlords from 12 to 57 — both were
publishing a near-empty map that read as if the machine had nothing to offer.
Gravitar (68), Space Duel (70), Fast Freddie (79) and Red Baron's Auxiliary
PCB (18) are new. Tempest gains 5.

Two results are worth more than the device count:

Red Baron's manual covers two PCBs whose designator grids collide — 8
collisions in TM-169, 6 in TM-171 — and locations() resolves a collision by
last write, so harvesting it whole would have merged two boards into one
wrong map without saying so. Split on the figure heading, both go to zero.
The Analog Vector-Generator half then agrees with Battlezone's hand-read game
PCB on 58 of the 63 positions they share, from sources with nothing in common:
six sides of DP-156 read by eye against OCR of two Red Baron parts lists. That
validates the hand read and the harvest at once. Gravitar and Space Duel check
each other the same way, 54 of 62, from different manuals.

The same split withdraws a claim. Red Baron's Auxiliary PCB is not
Battlezone's Auxiliary Math Box 035678-01: it agrees with it on 2 of 14 shared
designators and carries no Am2901 slices and no 82S129 microcode PROMs at all,
where the Math Box has four and six. A 555 sits where Battlezone has a bit
slice. The old note asserting a shared Math Box — and with it the claim that
Battlezone's signature codes apply to Red Baron — is withdrawn rather than
quietly edited, and what it implicates on the game PCB map is logged.

Everything else was already at its evidence limit: Crash 'n Score, Monte Carlo,
Asteroids Deluxe, Centipede, Football, Missile Command and the nine
single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
Parts:
- removed UA1, UB1, UE2, UN12, UR9: 74LS244, DIP-20_W7.62mm
- removed UA2: 74109, DIP-16_W7.62mm
- removed UA3, UE7, UH8, UN8, UN9: 74LS174, DIP-16_W7.62mm
- removed UA6, UE3, UN6: 74S04, DIP-14_W7.62mm
- removed UA7, UB5: 74LS02, DIP-14_W7.62mm
- removed UA8: 74LS109, DIP-16_W7.62mm
- removed UA9: 74LS164, DIP-14_W7.62mm
- removed UB3, UC1, UP7: 74LS139, DIP-16_W7.62mm
- removed UB6: 74LS27, DIP-14_W7.62mm
- removed UB7: 74S74, DIP-14_W7.62mm
- removed UB8, UD3: 74LS74, DIP-14_W7.62mm
- removed UB9, UC3, UR7: 74LS32, DIP-14_W7.62mm
- removed UC4: 74193, DIP-16_W7.62mm
- removed UD1: 136002-101, DIP-24_W15.24mm
- removed UD4: 74LS393, DIP-14_W7.62mm
- removed UD5, UD6: 74LS194, DIP-16_W7.62mm
- removed UD7: 136002-125, DIP-16_W7.62mm
- removed UE8, UF8: 74LS161, DIP-16_W7.62mm
- removed UF2: 74LS245, DIP-20_W7.62mm
- removed UF3: 74S08, DIP-14_W7.62mm
- removed UF6: 74S00, DIP-14_W7.62mm
- removed UH7, UJ3: 74LS175, DIP-16_W7.62mm
- removed UH9: 74LS399, DIP-16_W7.62mm
- removed UJ11: 74LS04, DIP-14_W7.62mm
- removed UL2, UM2, UN2, UP8: 74LS157, DIP-16_W7.62mm
- removed UL5: 74LS193, DIP-16_W7.62mm
- removed UL6: 74LS670, DIP-16_W7.62mm
- removed UL8: 74LS191, DIP-16_W7.62mm
- removed UN13: 8-position DIP switch, DIP-16_W7.62mm
- removed UN3: 136002-111, DIP-24_W15.24mm
- removed UN7: 74LS367, DIP-16_W7.62mm
- removed UR3: 136002-112, DIP-24_W15.24mm
- added UB10: 74LS245, DIP-20_W7.62mm, F.Cu at (254.6, 189.4)
- added UB13: 74LS367, DIP-16_W7.62mm, F.Cu at (330.8, 189.4)
- added UC10: 74LS367, DIP-16_W7.62mm, F.Cu at (254.6, 170.4)
- added UC13: 74LS367, DIP-16_W7.62mm, F.Cu at (330.8, 170.4)
- added UC9: 7408, DIP-14_W7.62mm, F.Cu at (229.2, 170.4)
- added UD12: 74LS20, DIP-14_W7.62mm, F.Cu at (305.4, 151.3)
- added UD13: 74LS139, DIP-16_W7.62mm, F.Cu at (330.8, 151.3)
- added UE10: 74LS02, DIP-14_W7.62mm, F.Cu at (254.6, 132.3)
- added UE13: 74LS157, DIP-16_W7.62mm, F.Cu at (330.8, 132.3)
- added UE14: 74LS157, DIP-16_W7.62mm, F.Cu at (356.2, 132.3)
- added UF10: 74LS157, DIP-16_W7.62mm, F.Cu at (254.6, 113.2)
- added UF11: 74LS367, DIP-16_W7.62mm, F.Cu at (280.0, 113.2)
- added UF12: 74LS367, DIP-16_W7.62mm, F.Cu at (305.4, 113.2)
- added UF14: 74LS32, DIP-14_W7.62mm, F.Cu at (356.2, 113.2)
- added UF15: 74LS194, DIP-16_W7.62mm, F.Cu at (381.6, 113.2)
- added UH1: 74LS161, DIP-16_W7.62mm, F.Cu at (26.0, 94.2)
- added UH10: 74LS245, DIP-20_W7.62mm, F.Cu at (254.6, 94.2)
- added UH11: 74LS245, DIP-20_W7.62mm, F.Cu at (280.0, 94.2)
- added UH14: 74LS157, DIP-16_W7.62mm, F.Cu at (356.2, 94.2)
- added UH15: 74LS194, DIP-16_W7.62mm, F.Cu at (381.6, 94.2)
- added UJ12: 74LS273, DIP-20_W7.62mm, F.Cu at (305.4, 75.2)
- added UJ9: 74LS273, DIP-20_W7.62mm, F.Cu at (229.2, 75.2)
- added UK1: 74LS161, DIP-16_W7.62mm, F.Cu at (26.0, 56.1)
- added UK10: 74LS163, DIP-16_W7.62mm, F.Cu at (254.6, 56.1)
- added UK12: 74LS20, DIP-14_W7.62mm, F.Cu at (305.4, 56.1)
- added UK13: 74LS157, DIP-16_W7.62mm, F.Cu at (330.8, 56.1)
- added UK3: 74LS32, DIP-14_W7.62mm, F.Cu at (76.8, 56.1)
- added UK4: 74LS32, DIP-14_W7.62mm, F.Cu at (102.2, 56.1)
- added UL1: 74LS161, DIP-16_W7.62mm, F.Cu at (26.0, 37.0)
- added UL13: 74LS157, DIP-16_W7.62mm, F.Cu at (330.8, 37.0)
- added UL3: 74LS74, DIP-14_W7.62mm, F.Cu at (76.8, 37.0)
- added UL4: 74LS174, DIP-16_W7.62mm, F.Cu at (102.2, 37.0)
- added UM10: 74LS163, DIP-16_W7.62mm, F.Cu at (254.6, 18.0)
- added UM11: 74LS157, DIP-16_W7.62mm, F.Cu at (280.0, 18.0)
- added UM13: 74LS157, DIP-16_W7.62mm, F.Cu at (330.8, 18.0)
- added UM3: 74LS02, DIP-14_W7.62mm, F.Cu at (76.8, 18.0)
- added UM4: 74LS32, DIP-14_W7.62mm, F.Cu at (102.2, 18.0)
- added UM7: 74LS00, DIP-14_W7.62mm, F.Cu at (178.4, 18.0)
- added UM8: 74LS08, DIP-14_W7.62mm, F.Cu at (203.8, 18.0)
- added UM9: 74LS86, DIP-14_W7.62mm, F.Cu at (229.2, 18.0)
- UA4: value 74LS08 -> 74LS02
- UB4: value 74LS393 -> 74LS08
- UC2: value 90-6013 -> 74LS245; footprint DIP-40_W15.24mm -> DIP-20_W7.62mm
- UC5: value 74S260 -> 74LS367; footprint DIP-14_W7.62mm -> DIP-16_W7.62mm
- UC6: value 74S02 -> 74LS367; footprint DIP-14_W7.62mm -> DIP-16_W7.62mm
- UC7: value 74S74 -> 74LS273; footprint DIP-14_W7.62mm -> DIP-20_W7.62mm
- UC8: value 74LS161 -> 74LS393; footprint DIP-16_W7.62mm -> DIP-14_W7.62mm
- UD10: value DAC-08 -> 74LS259
- UD8: value 74LS161 -> 74LS175
- UD9: value 74LS273 -> 74LS08; footprint DIP-20_W7.62mm -> DIP-14_W7.62mm
- UE4: value 74LS161 -> 74LS367
- UE5: value 74LS194 -> 74LS367
- UE6: value 74LS14 -> 74LS86
- UE9: value 74LS20 -> 74LS74
- UF4: value 74LS10 -> 74LS74
- UF5: value 74LS194 -> 74LS74; footprint DIP-16_W7.62mm -> DIP-14_W7.62mm
- UF7: value 74LS42 -> 74LS00; footprint DIP-16_W7.62mm -> DIP-14_W7.62mm
- UH2: value 74LS245 -> 74LS161; footprint DIP-20_W7.62mm -> DIP-16_W7.62mm
- UH3: value 74LS245 -> 74LS74; footprint DIP-20_W7.62mm -> DIP-14_W7.62mm
- UH4: value 74LS174 -> 74LS74; footprint DIP-16_W7.62mm -> DIP-14_W7.62mm
- UH5: value 74LS194 -> 74LS86; footprint DIP-16_W7.62mm -> DIP-14_W7.62mm
- UH6: value 74LS194 -> 74LS32; footprint DIP-16_W7.62mm -> DIP-14_W7.62mm
- UJ4: value 74LS02 -> 74LS00
- UJ5: value 74LS139 -> 74LS86; footprint DIP-16_W7.62mm -> DIP-14_W7.62mm
- UJ6: value 74LS191 -> 74LS02; footprint DIP-16_W7.62mm -> DIP-14_W7.62mm
- UJ7: value 74LS175 -> 74LS157
- UJ8: value 74LS32 -> 74LS157; footprint DIP-14_W7.62mm -> DIP-16_W7.62mm
- UK11: value TL082 -> 74LS157; footprint DIP-8_W7.62mm -> DIP-16_W7.62mm
- UK2: value 74LS157 -> 74LS86; footprint DIP-16_W7.62mm -> DIP-14_W7.62mm
- UK5, UM5: value 74LS193 -> 74LS20; footprint DIP-16_W7.62mm -> DIP-14_W7.62mm
- UK6: value 74LS670 -> 74LS00; footprint DIP-16_W7.62mm -> DIP-14_W7.62mm
- UK7: value 74LS367 -> 74LS08; footprint DIP-16_W7.62mm -> DIP-14_W7.62mm
- UK8: value 74LS175 -> 74LS273; footprint DIP-16_W7.62mm -> DIP-20_W7.62mm
- UK9: value 74LS00 -> 74LS86
- UL12: value 8-position DIP switch -> 74LS273; footprint DIP-16_W7.62mm -> DIP-20_W7.62mm
- UM12: value 74LS244 -> 74LS86; footprint DIP-20_W7.62mm -> DIP-14_W7.62mm
- UM6: value 74LS670 -> 74LS20; footprint DIP-16_W7.62mm -> DIP-14_W7.62mm
- moved UB4 57.2 mm to (102.2, 189.4)
- moved UC2 57.2 mm to (51.4, 170.4)
- moved UC5 57.2 mm to (127.6, 170.4)
- moved UC6 57.2 mm to (153.0, 170.4)
- moved UC7 57.2 mm to (178.4, 170.4)
- moved UC8 57.2 mm to (203.8, 170.4)
- moved UD10 57.2 mm to (254.6, 151.3)
- moved UD8 57.2 mm to (203.8, 151.3)
- moved UD9 57.2 mm to (229.2, 151.3)
- moved UF4 57.2 mm to (102.2, 113.2)
- moved UF5 57.2 mm to (127.6, 113.2)
- moved UF7 57.2 mm to (178.4, 113.2)
- moved UJ2 57.2 mm to (51.4, 75.2)
- moved UJ4 57.2 mm to (102.2, 75.2)
- moved UJ5 57.2 mm to (127.6, 75.2)
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Other:
- board size 300 x 300 mm -> 417 x 238 mm
