File: kicad/gravitar/gravitar.kicad_pcb (KiCad board)
At the start: 2 copper layers, 300 x 300 mm, 57 parts

Commit message: Fill four thin boards and add four more, from the parts lists
The parts-list harvest was described as swept. It was swept for finding new
machines to hand-read; it had not been run against the boards already here.
Running it over all 2,389 cached documents finds 29 boards where there was
one, and 1,864 devices where there were 1,365.

Red Baron goes from 15 devices to 66 and Warlords from 12 to 57 — both were
publishing a near-empty map that read as if the machine had nothing to offer.
Gravitar (68), Space Duel (70), Fast Freddie (79) and Red Baron's Auxiliary
PCB (18) are new. Tempest gains 5.

Two results are worth more than the device count:

Red Baron's manual covers two PCBs whose designator grids collide — 8
collisions in TM-169, 6 in TM-171 — and locations() resolves a collision by
last write, so harvesting it whole would have merged two boards into one
wrong map without saying so. Split on the figure heading, both go to zero.
The Analog Vector-Generator half then agrees with Battlezone's hand-read game
PCB on 58 of the 63 positions they share, from sources with nothing in common:
six sides of DP-156 read by eye against OCR of two Red Baron parts lists. That
validates the hand read and the harvest at once. Gravitar and Space Duel check
each other the same way, 54 of 62, from different manuals.

The same split withdraws a claim. Red Baron's Auxiliary PCB is not
Battlezone's Auxiliary Math Box 035678-01: it agrees with it on 2 of 14 shared
designators and carries no Am2901 slices and no 82S129 microcode PROMs at all,
where the Math Box has four and six. A 555 sits where Battlezone has a bit
slice. The old note asserting a shared Math Box — and with it the claim that
Battlezone's signature codes apply to Red Baron — is withdrawn rather than
quietly edited, and what it implicates on the game PCB map is logged.

Everything else was already at its evidence limit: Crash 'n Score, Monte Carlo,
Asteroids Deluxe, Centipede, Football, Missile Command and the nine
single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
Parts:
- removed UB5: 74LS90, DIP-14_W7.62mm
- removed UB6: 74LS04, DIP-14_W7.62mm
- removed UC3: 74LS139, DIP-16_W7.62mm
- removed UC4: 74LS00, DIP-14_W7.62mm
- removed UC5: 74LS10, DIP-14_W7.62mm
- removed UD3: 74LS42, DIP-16_W7.62mm
- removed UD4: 74LS32, DIP-14_W7.62mm
- removed UD5, UD8: 74LS174, DIP-16_W7.62mm
- removed UF5: 74LS83, DIP-16_W7.62mm
- removed UK4, UM4, UP7: 74LS153, DIP-16_W7.62mm
- removed UK7, UP5: 74LS163A, DIP-16_W7.62mm
- removed UL2: 74LS257, DIP-16_W7.62mm
- removed UL7: 74LS273, DIP-20_W7.62mm
- removed UN4: 74LS74, DIP-14_W7.62mm
- removed UP3: 74S04, DIP-14_W7.62mm
- removed UP9: 74LS259, DIP-16_W7.62mm
- added UA4: 555, DIP-8_W7.62mm, F.Cu at (102.2, 265.6)
- added UA6: 74S74, DIP-14_W7.62mm, F.Cu at (153.0, 265.6)
- added UA7: 74S74, DIP-14_W7.62mm, F.Cu at (178.4, 265.6)
- added UA8: 74LS194, DIP-16_W7.62mm, F.Cu at (203.8, 265.6)
- added UB8: 74LS194, DIP-16_W7.62mm, F.Cu at (203.8, 246.6)
- added UC8: 74LS194, DIP-16_W7.62mm, F.Cu at (203.8, 227.6)
- added UE6: 74LS175, DIP-16_W7.62mm, F.Cu at (153.0, 189.4)
- added UE8: 74LS273, DIP-20_W7.62mm, F.Cu at (203.8, 189.4)
- added UF6: 74LS157, DIP-16_W7.62mm, F.Cu at (153.0, 170.4)
- added UH2: 74LS244, DIP-20_W7.62mm, F.Cu at (51.4, 151.3)
- added UH3: 74LS20, DIP-14_W7.62mm, F.Cu at (76.8, 151.3)
- added UH5: 74LS20, DIP-14_W7.62mm, F.Cu at (127.6, 151.3)
- added UH6: 74LS175, DIP-16_W7.62mm, F.Cu at (153.0, 151.3)
- added UJ2: 74LS374, DIP-20_W7.62mm, F.Cu at (51.4, 132.3)
- added UJ5: 74S260, DIP-14_W7.62mm, F.Cu at (127.6, 132.3)
- added UK10: 74LS175, DIP-16_W7.62mm, F.Cu at (254.6, 113.2)
- added UK3: 74LS74, DIP-14_W7.62mm, F.Cu at (76.8, 113.2)
- added UK5: 74LS02, DIP-14_W7.62mm, F.Cu at (127.6, 113.2)
- added UK8: 74LS157, DIP-16_W7.62mm, F.Cu at (203.8, 113.2)
- added UL3: 74LS00, DIP-14_W7.62mm, F.Cu at (76.8, 94.2)
- added UL5: 74LS74, DIP-14_W7.62mm, F.Cu at (127.6, 94.2)
- added UL8: 74LS157, DIP-16_W7.62mm, F.Cu at (203.8, 94.2)
- added UL9: 74LS244, DIP-20_W7.62mm, F.Cu at (229.2, 94.2)
- added UM9: 74LS244, DIP-20_W7.62mm, F.Cu at (229.2, 75.2)
- added UN3: 74LS157, DIP-16_W7.62mm, F.Cu at (76.8, 56.1)
- added UP2: 74LS174, DIP-16_W7.62mm, F.Cu at (51.4, 37.0)
- added UP8: 74LS245, DIP-20_W7.62mm, F.Cu at (203.8, 37.0)
- added UR3: 74LS157, DIP-16_W7.62mm, F.Cu at (76.8, 18.0)
- added UR4: 74LS32, DIP-14_W7.62mm, F.Cu at (102.2, 18.0)
- added UR6: 74LS161, DIP-16_W7.62mm, F.Cu at (153.0, 18.0)
- added UR9: 74LS273, DIP-20_W7.62mm, F.Cu at (229.2, 18.0)
- UB7: value 74LS74 -> 74S02
- UC6: value 74LS157 -> 74LS175
- UC7: value 74LS08 -> 74LS191; footprint DIP-14_W7.62mm -> DIP-16_W7.62mm
- UD6: value 74LS86 -> 74LS175; footprint DIP-14_W7.62mm -> DIP-16_W7.62mm
- UD7: value 74LS166 -> 74LS175
- UE2: value 74LS245 -> 74LS244
- UE4: value 74LS32 -> 74193; footprint DIP-14_W7.62mm -> DIP-16_W7.62mm
- UE5: value 74LS83 -> 74109
- UE7: value 74LS157 -> 74S00; footprint DIP-16_W7.62mm -> DIP-14_W7.62mm
- UF2: value 74LS373 -> 74LS245
- UF3: value 74LS10 -> 74S04
- UF4: value 74LS273 -> 74LS393; footprint DIP-20_W7.62mm -> DIP-14_W7.62mm
- UF7: value 74LS157 -> 74LS14; footprint DIP-16_W7.62mm -> DIP-14_W7.62mm
- UF8, UH8: value 74LS257 -> 74LS194
- UH4: value 74LS153 -> 74LS393; footprint DIP-16_W7.62mm -> DIP-14_W7.62mm
- UH7: value 74LS157 -> 74LS42
- UJ4: value 74LS153 -> 74LS161
- UJ6: value 74LS04 -> 74LS32
- UJ7: value 74LS157 -> 74LS139
- UJ8: value 74LS166 -> 74LS194
- UK2: value 74LS257 -> 74LS175
- UK6: value 74LS74 -> 74LS02
- UL4: value 74LS153 -> 74LS08; footprint DIP-16_W7.62mm -> DIP-14_W7.62mm
- UL6: value 74LS175 -> 74LS08; footprint DIP-16_W7.62mm -> DIP-14_W7.62mm
- UM3: value 74LS257 -> 74LS164; footprint DIP-16_W7.62mm -> DIP-14_W7.62mm
- UM5: value 74LS257 -> 74LS32; footprint DIP-16_W7.62mm -> DIP-14_W7.62mm
- UM6: value 82S129 -> 74LS161
- UM8: value 74LS163A -> 74LS157
- UN5: value 74LS163A -> 74LS02; footprint DIP-16_W7.62mm -> DIP-14_W7.62mm
- UN6, UP6: value 74LS163A -> 74LS161
- UN8: value 74S74 -> 74LS157; footprint DIP-14_W7.62mm -> DIP-16_W7.62mm
- UN9: value 74LS32 -> 74LS244; footprint DIP-14_W7.62mm -> DIP-20_W7.62mm
- UP4: value 74LS163A -> 74LS174
Other:
- board size 300 x 300 mm -> 290 x 295 mm
