File: kicad/space-duel/space-duel.kicad_pcb (KiCad board)
At the start: 2 copper layers, 300 x 300 mm, 93 parts

Commit message: Fill four thin boards and add four more, from the parts lists
The parts-list harvest was described as swept. It was swept for finding new
machines to hand-read; it had not been run against the boards already here.
Running it over all 2,389 cached documents finds 29 boards where there was
one, and 1,864 devices where there were 1,365.

Red Baron goes from 15 devices to 66 and Warlords from 12 to 57 — both were
publishing a near-empty map that read as if the machine had nothing to offer.
Gravitar (68), Space Duel (70), Fast Freddie (79) and Red Baron's Auxiliary
PCB (18) are new. Tempest gains 5.

Two results are worth more than the device count:

Red Baron's manual covers two PCBs whose designator grids collide — 8
collisions in TM-169, 6 in TM-171 — and locations() resolves a collision by
last write, so harvesting it whole would have merged two boards into one
wrong map without saying so. Split on the figure heading, both go to zero.
The Analog Vector-Generator half then agrees with Battlezone's hand-read game
PCB on 58 of the 63 positions they share, from sources with nothing in common:
six sides of DP-156 read by eye against OCR of two Red Baron parts lists. That
validates the hand read and the harvest at once. Gravitar and Space Duel check
each other the same way, 54 of 62, from different manuals.

The same split withdraws a claim. Red Baron's Auxiliary PCB is not
Battlezone's Auxiliary Math Box 035678-01: it agrees with it on 2 of 14 shared
designators and carries no Am2901 slices and no 82S129 microcode PROMs at all,
where the Math Box has four and six. A 555 sits where Battlezone has a bit
slice. The old note asserting a shared Math Box — and with it the claim that
Battlezone's signature codes apply to Red Baron — is withdrawn rather than
quietly edited, and what it implicates on the game PCB map is logged.

Everything else was already at its evidence limit: Crash 'n Score, Monte Carlo,
Asteroids Deluxe, Centipede, Football, Missile Command and the nine
single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
Parts:
- removed UA1, UM12, UN12: 74LS244, DIP-20_W7.62mm
- removed UA2: 74109, DIP-16_W7.62mm
- removed UA3: 74LS174, DIP-16_W7.62mm
- removed UA6: 74S04, DIP-14_W7.62mm
- removed UA9: 74LS164, DIP-14_W7.62mm
- removed UB3, UP7: 74LS139, DIP-16_W7.62mm
- removed UB4, UD4: 74LS393, DIP-14_W7.62mm
- removed UB5: 74LS02, DIP-14_W7.62mm
- removed UB6: 74LS27, DIP-14_W7.62mm
- removed UB7: 74S74, DIP-14_W7.62mm
- removed UB9, UC3, UR7: 74LS32, DIP-14_W7.62mm
- removed UC2: 90-6013, DIP-40_W15.24mm
- removed UC4: 74193, DIP-16_W7.62mm
- removed UC5: 74S260, DIP-14_W7.62mm
- removed UD1: 136002-101, DIP-24_W15.24mm
- removed UD10: DAC-08, DIP-16_W7.62mm
- removed UD3: 74LS74, DIP-14_W7.62mm
- removed UD5, UF5: 74LS194, DIP-16_W7.62mm
- removed UD8, UE8: 74LS161, DIP-16_W7.62mm
- removed UD9: 74LS273, DIP-20_W7.62mm
- removed UE9: 74LS20, DIP-14_W7.62mm
- removed UH9: 74LS399, DIP-16_W7.62mm
- removed UJ11: 74LS04, DIP-14_W7.62mm
- removed UJ7: 74LS175, DIP-16_W7.62mm
- removed UK11: TL082, DIP-8_W7.62mm
- removed UK7, UN7: 74LS367, DIP-16_W7.62mm
- removed UL12, UN13: 8-position DIP switch, DIP-16_W7.62mm
- removed UL2, UM2, UN2: 74LS157, DIP-16_W7.62mm
- added UK10: 74LS175, DIP-16_W7.62mm, F.Cu at (254.6, 113.2)
- added UK3: 74LS74, DIP-14_W7.62mm, F.Cu at (76.8, 113.2)
- added UK4: 74LS10, DIP-14_W7.62mm, F.Cu at (102.2, 113.2)
- added UL10: 7433, DIP-14_W7.62mm, F.Cu at (254.6, 94.2)
- added UL3: 74LS00, DIP-14_W7.62mm, F.Cu at (76.8, 94.2)
- added UL4: 74LS42, DIP-16_W7.62mm, F.Cu at (102.2, 94.2)
- added UL9: 74LS251, DIP-16_W7.62mm, F.Cu at (229.2, 94.2)
- added UM3: 74LS164, DIP-14_W7.62mm, F.Cu at (76.8, 75.2)
- added UM4: 74LS27, DIP-14_W7.62mm, F.Cu at (102.2, 75.2)
- added UM8: 74LS157, DIP-16_W7.62mm, F.Cu at (203.8, 75.2)
- added UM9: 74LS244, DIP-20_W7.62mm, F.Cu at (229.2, 75.2)
- added UP2: 74LS174, DIP-16_W7.62mm, F.Cu at (51.4, 37.0)
- added UP3: 74LS42, DIP-16_W7.62mm, F.Cu at (76.8, 37.0)
- added UP6: 74LS161, DIP-16_W7.62mm, F.Cu at (153.0, 37.0)
- added UR2: 74LS42, DIP-16_W7.62mm, F.Cu at (51.4, 18.0)
- added UR4: 74LS174, DIP-16_W7.62mm, F.Cu at (102.2, 18.0)
- added UR6: 74LS161, DIP-16_W7.62mm, F.Cu at (153.0, 18.0)
- UA4: value 74LS08 -> 555; footprint DIP-14_W7.62mm -> DIP-8_W7.62mm
- UA7: value 74LS02 -> 74LS74
- UA8: value 74LS109 -> 74LS194
- UB8: value 74LS74 -> 74LS194; footprint DIP-14_W7.62mm -> DIP-16_W7.62mm
- UC1: value 74LS139 -> 74LS244; footprint DIP-16_W7.62mm -> DIP-20_W7.62mm
- UC6: value 74S02 -> 74LS175; footprint DIP-14_W7.62mm -> DIP-16_W7.62mm
- UC7: value 74S74 -> 74LS191; footprint DIP-14_W7.62mm -> DIP-16_W7.62mm
- UC8, UF8: value 74LS161 -> 74LS194
- UD6, UH6: value 74LS194 -> 74LS175
- UD7: value 136002-125 -> 74LS175
- UE3: value 74S04 -> 74LS00
- UE4: value 74LS161 -> 74193
- UE5: value 74LS194 -> 74LS109
- UE6: value 74LS14 -> 74LS175; footprint DIP-14_W7.62mm -> DIP-16_W7.62mm
- UE7: value 74LS174 -> 74S00; footprint DIP-16_W7.62mm -> DIP-14_W7.62mm
- UF3: value 74S08 -> 74S04
- UF4: value 74LS10 -> 74LS393
- UF6: value 74S00 -> 74LS157; footprint DIP-14_W7.62mm -> DIP-16_W7.62mm
- UF7: value 74LS42 -> 74LS14; footprint DIP-16_W7.62mm -> DIP-14_W7.62mm
- UH2: value 74LS245 -> 74LS244
- UH3: value 74LS245 -> 74LS02; footprint DIP-20_W7.62mm -> DIP-14_W7.62mm
- UH4: value 74LS174 -> 74LS393; footprint DIP-16_W7.62mm -> DIP-14_W7.62mm
- UH5: value 74LS194 -> 74LS20; footprint DIP-16_W7.62mm -> DIP-14_W7.62mm
- UH7: value 74LS175 -> 74LS42
- UH8: value 74LS174 -> 74LS194
- UJ2: value 74LS139 -> 74LS374; footprint DIP-16_W7.62mm -> DIP-20_W7.62mm
- UJ3: value 74LS175 -> 74LS04; footprint DIP-16_W7.62mm -> DIP-14_W7.62mm
- UJ4: value 74LS02 -> 74LS161; footprint DIP-14_W7.62mm -> DIP-16_W7.62mm
- UJ5: value 74LS139 -> 74S260; footprint DIP-16_W7.62mm -> DIP-14_W7.62mm
- UJ6: value 74LS191 -> 74LS32; footprint DIP-16_W7.62mm -> DIP-14_W7.62mm
- UJ8: value 74LS32 -> 74LS194; footprint DIP-14_W7.62mm -> DIP-16_W7.62mm
- UK2: value 74LS157 -> 74LS175
- UK5: value 74LS193 -> 74LS02; footprint DIP-16_W7.62mm -> DIP-14_W7.62mm
- UK6: value 74LS670 -> 74LS139
- UK8: value 74LS175 -> 74LS157
- UK9: value 74LS00 -> 74LS04
- UL5: value 74LS193 -> 74LS74; footprint DIP-16_W7.62mm -> DIP-14_W7.62mm
- UL6: value 74LS670 -> 74LS08; footprint DIP-16_W7.62mm -> DIP-14_W7.62mm
- UL8: value 74LS191 -> 74LS157
- UM5: value 74LS193 -> 74LS32; footprint DIP-16_W7.62mm -> DIP-14_W7.62mm
- UM6: value 74LS670 -> 74LS161
- UN3: value 136002-111 -> 74LS32; footprint DIP-24_W15.24mm -> DIP-14_W7.62mm
- UN6: value 74S04 -> 74LS161; footprint DIP-14_W7.62mm -> DIP-16_W7.62mm
- UN8: value 74LS174 -> 74LS157
- UN9: value 74LS174 -> 74LS251
- UP8: value 74LS157 -> 74LS245; footprint DIP-16_W7.62mm -> DIP-20_W7.62mm
- UR3: value 136002-112 -> 74LS08; footprint DIP-24_W15.24mm -> DIP-14_W7.62mm
- UR9: value 74LS244 -> 74LS273
- moved UB1 9.53 mm to (26.0, 246.6)
- moved UN3 9.52 mm to (76.8, 56.1)
Other:
- board size 300 x 300 mm -> 290 x 295 mm
