File: kicad/indy-4/indy-4.kicad_pcb (KiCad board)
At the start: 2 copper layers, 198.4 x 228.5 mm, 30 parts

Commit message: Drop a cell both readings claim, instead of taking the last one
locations() detects a designator claimed twice by the same parts list and
returns the collision alongside the mapping. harvest() took only
locations(...)[0] and dropped that half of the answer on the floor, so a
contested cell was resolved by whichever reading came last in the file.

22 devices on the published site were chosen that way: Food Fight 1, I-Robot 8,
Indy 4 3, Monte Carlo 4, Pole Position 6. They are withdrawn. merge only ever
adds cells, so re-running it could not undo them — they had to come off
explicitly. Both readings are recorded in each board's read file rather than
just deleted, because a repairer at the bench is better served by "it is one of
these two" than by a silent gap.

A contested cell is now kept only when every reading of it names the same
device — '74L886' against '74LS86' is one part and an OCR of S as 8, and Orbit's
three such cells stay. Anything else is dropped and printed.

It deliberately does NOT use plausible() to break the tie, though the
cross-printing split does. plausible() does not recognise the Fairchild 93xx and
96xx series: it calls 9312, 9322 and 9602 implausible, and 9316 too — which this
repo's own equivalence table documents as Fairchild's 74161. Filtering on it here
would have discarded the 9312 reading of Indy 4's B3 and "resolved" that cell to
a 7474, a different device entirely. A false correction is worse than the
collision it replaces. The split path has the same blind spot and is now flagged
in HANDOFF, unaudited.

The fix also unblocks the two boards withheld last time for exactly this reason.
Pole Position II (38 devices, 8 cells dropped) and Xevious (18, 1 dropped) no
longer need figure-splitting to be safe, because a cell nothing can attribute is
now simply absent rather than guessed.

47 boards, 2,489 devices.

Co-Authored-By: Claude Opus 5 <noreply@anthropic.com>
Parts:
- removed UA3: 7493, DIP-14_W7.62mm
- removed UB3: 9312, DIP-16_W7.62mm
- removed UH2: 9322, DIP-16_W7.62mm
