File: kicad/pole-position-2/pole-position-2.kicad_pcb (KiCad board)
At the start: 2 copper layers, 366 x 257 mm, 49 parts, among them U10B 74LS74, U10D 74LS174, U10E 74LS257, U10N 74LS85, U11B 74107, U11C 7497, U11F 74LS174, U11H 74LS174, U11K 74LS139, U12C 74LS161, U12D 74LS393, U12F 74LS86, U13F 74LS20, U1B 74107, U2E 74LS74, U2H 74LS139, U3H 74LS175, U4B 74LS367, U4C 74LS373, U4H 74LS157, U4K 74LS174, U4M 74LS373, U5A 74LS74, U5B 74LS174, U5C 74LS174, U5F 74LS245, U5H 74LS175, U5K 74LS244, U5N 74LS74, U6H 74LS245, U6L 74LS109, U7C 74S04, U7D 74LS32, U7L 74LS273, U7M 74LS273, U7N 74S04, U8B 74S00, U8C 74LS157, U8E 74LS259, U8F 74LS367, U8K 4066, U8M 74LS04, U9B 74LS20, U9C 74LS157, U9E 74LS257, U9H 74LS161, U9K 7497, U9L 74LS174, U9N 74LS85

Commit message: Drop a cell both readings claim, instead of taking the last one
locations() detects a designator claimed twice by the same parts list and
returns the collision alongside the mapping. harvest() took only
locations(...)[0] and dropped that half of the answer on the floor, so a
contested cell was resolved by whichever reading came last in the file.

22 devices on the published site were chosen that way: Food Fight 1, I-Robot 8,
Indy 4 3, Monte Carlo 4, Pole Position 6. They are withdrawn. merge only ever
adds cells, so re-running it could not undo them — they had to come off
explicitly. Both readings are recorded in each board's read file rather than
just deleted, because a repairer at the bench is better served by "it is one of
these two" than by a silent gap.

A contested cell is now kept only when every reading of it names the same
device — '74L886' against '74LS86' is one part and an OCR of S as 8, and Orbit's
three such cells stay. Anything else is dropped and printed.

It deliberately does NOT use plausible() to break the tie, though the
cross-printing split does. plausible() does not recognise the Fairchild 93xx and
96xx series: it calls 9312, 9322 and 9602 implausible, and 9316 too — which this
repo's own equivalence table documents as Fairchild's 74161. Filtering on it here
would have discarded the 9312 reading of Indy 4's B3 and "resolved" that cell to
a 7474, a different device entirely. A false correction is worse than the
collision it replaces. The split path has the same blind spot and is now flagged
in HANDOFF, unaudited.

The fix also unblocks the two boards withheld last time for exactly this reason.
Pole Position II (38 devices, 8 cells dropped) and Xevious (18, 1 dropped) no
longer need figure-splitting to be safe, because a cell nothing can attribute is
now simply absent rather than guessed.

47 boards, 2,489 devices.

Co-Authored-By: Claude Opus 5 <noreply@anthropic.com>
Parts:
- removed U10D, U11F, U4K, U9L: 74LS174, DIP-16_W7.62mm
- removed the U10E at (254.6, 151.3)
- removed U10N, U9N: 74LS85, DIP-16_W7.62mm
- removed U11B, U1B: 74107, DIP-14_W7.62mm
- removed U11C, U9K: 7497, DIP-16_W7.62mm
- removed the U11H at (280.0, 113.2)
- removed U11K, U2H: 74LS139, DIP-16_W7.62mm
- removed U12C: 74LS161, DIP-16_W7.62mm
- removed U13F, U9B: 74LS20, DIP-14_W7.62mm
- removed the U2E at (51.4, 151.3)
- removed U3H, U5H: 74LS175, DIP-16_W7.62mm
- removed U4B: 74LS367, DIP-16_W7.62mm
- removed the U4C at (102.2, 189.4)
- removed U4H, U8C, U9C: 74LS157, DIP-16_W7.62mm
- removed U4M: 74LS373, DIP-20_W7.62mm
- removed U5A, U5N: 74LS74, DIP-14_W7.62mm
- removed U5F, U6H: 74LS245, DIP-20_W7.62mm
- removed U5K: 74LS244, DIP-20_W7.62mm
- removed U6L: 74LS109, DIP-16_W7.62mm
- removed U7C, U7N: 74S04, DIP-14_W7.62mm
- removed U7D: 74LS32, DIP-14_W7.62mm
- removed the U7L at (178.4, 56.1)
- removed the U7M at (178.4, 37.0)
- removed U8E: 74LS259, DIP-16_W7.62mm
- removed the U8F at (203.8, 132.3)
- removed U8K: 4066, DIP-14_W7.62mm
- removed U9E: 74LS257, DIP-16_W7.62mm
- added U10E: 74LS08, DIP-14_W7.62mm, F.Cu at (254.6, 132.3)
- added U10F: 74S04, DIP-14_W7.62mm, F.Cu at (254.6, 113.2)
- added U10H: 74LS157, DIP-16_W7.62mm, F.Cu at (254.6, 94.2)
- added U10J: 74LS157, DIP-16_W7.62mm, F.Cu at (254.6, 75.2)
- added U10K: 4066, DIP-14_W7.62mm, F.Cu at (254.6, 56.1)
- added U10L: 4066, DIP-14_W7.62mm, F.Cu at (254.6, 37.0)
- added U11D: 74LS174, DIP-16_W7.62mm, F.Cu at (280.0, 151.3)
- added U11H: 74S00, DIP-14_W7.62mm, F.Cu at (280.0, 94.2)
- added U11M: 4066, DIP-14_W7.62mm, F.Cu at (280.0, 18.0)
- added U1H: 74S04, DIP-14_W7.62mm, F.Cu at (26.0, 94.2)
- added U1K: 74LS85, DIP-16_W7.62mm, F.Cu at (26.0, 56.1)
- added U2A: 7497, DIP-16_W7.62mm, F.Cu at (51.4, 208.5)
- added U2E: 74LS273, DIP-20_W7.62mm, F.Cu at (51.4, 132.3)
- added U2F: 74LS273, DIP-20_W7.62mm, F.Cu at (51.4, 113.2)
- added U3F: 74LS273, DIP-20_W7.62mm, F.Cu at (76.8, 113.2)
- added U4C: 74LS174, DIP-16_W7.62mm, F.Cu at (102.2, 170.4)
- added U4J: 7497, DIP-16_W7.62mm, F.Cu at (102.2, 75.2)
- added U4L: 74LS139, DIP-16_W7.62mm, F.Cu at (102.2, 37.0)
- added U6C: 74LS157, DIP-16_W7.62mm, F.Cu at (153.0, 170.4)
- added U6F: 74LS367, DIP-16_W7.62mm, F.Cu at (153.0, 113.2)
- added U6K: 74LS161, DIP-16_W7.62mm, F.Cu at (153.0, 56.1)
- added U6M: 74LS00, DIP-14_W7.62mm, F.Cu at (153.0, 18.0)
- added U7E: 74LS245, DIP-20_W7.62mm, F.Cu at (178.4, 132.3)
- added U7L: 74LS174, DIP-16_W7.62mm, F.Cu at (178.4, 37.0)
- added U7M: 74LS86, DIP-14_W7.62mm, F.Cu at (178.4, 18.0)
- added U8A: 74LS74, DIP-14_W7.62mm, F.Cu at (203.8, 208.5)
- added U8D: 74LS245, DIP-20_W7.62mm, F.Cu at (203.8, 151.3)
- added U8F: 4066, DIP-14_W7.62mm, F.Cu at (203.8, 113.2)
- added U8J: 74LS257, DIP-16_W7.62mm, F.Cu at (203.8, 75.2)
- added U8L: 4584B, DIP-14_W7.62mm, F.Cu at (203.8, 37.0)
- U10B: value 74LS74 -> 4066
- U12F: value 74LS86 -> 74S04
- U8M: value 74LS04 -> 74S04
- U9H: value 74LS161 -> 74LS157
- moved U10B 19.1 mm to (254.6, 189.4)
- moved U12D 19.1 mm to (305.4, 151.3)
- moved U12F 19.1 mm to (305.4, 113.2)
- moved U5B 19.1 mm to (127.6, 189.4)
- moved U8B 19.1 mm to (203.8, 189.4)
- moved U8M 19.0 mm to (203.8, 18.0)
- moved U9H 19.0 mm to (229.2, 94.2)
- moved U5C 19.0 mm to (127.6, 170.4)
Other:
- board size 366 x 257 mm -> 341 x 238 mm
