File: kicad/i-robot/i-robot.kicad_pcb (KiCad board)
At the start: 2 copper layers, 544 x 276 mm, 53 parts, among them U10A 74S157, U10B 74S00, U10D 74S32, U10F 74S10, U10K 74LS244, U10L 74LS273, U10P 74S04, U12E 74153, U12P 74S00, U13K 74LS174, U13L 74LS174, U1A 74LS157, U1B 74LS244, U20D 74LS273, U2F 74LS244, U2H 74LS374, U2L 74LS157, U2M 74LS374, U3B 74LS08, U3H 74LS257, U3K 74S32, U3L 74LS257, U3N 74S08, U3P 74LS244, U4A 74LS139, U4H 74LS244, U4P 74LS27, U5A 74LS00, U5K 74S157, U5L 74S157, U5R 74S04, U6A 74LS14, U6B 74LS04, U6D 74LS74, U7C 74LS139, U7D 74LS139, U7K 74LS163A, U7L 74S08, U8B 74LS139, U8D 74LS08, U8F 74S04, U8H 74LS125, U8K 74LS83, U8L 74S163, U8M 74LS04, U8N 74LS00, U8P 74LS74, U8R 74S08, U9A 74LS374, U9B 74LS374, U9C 74LS85, U9D 74LS85, U9K 74LS273

Commit message: Drop a cell both readings claim, instead of taking the last one
locations() detects a designator claimed twice by the same parts list and
returns the collision alongside the mapping. harvest() took only
locations(...)[0] and dropped that half of the answer on the floor, so a
contested cell was resolved by whichever reading came last in the file.

22 devices on the published site were chosen that way: Food Fight 1, I-Robot 8,
Indy 4 3, Monte Carlo 4, Pole Position 6. They are withdrawn. merge only ever
adds cells, so re-running it could not undo them — they had to come off
explicitly. Both readings are recorded in each board's read file rather than
just deleted, because a repairer at the bench is better served by "it is one of
these two" than by a silent gap.

A contested cell is now kept only when every reading of it names the same
device — '74L886' against '74LS86' is one part and an OCR of S as 8, and Orbit's
three such cells stay. Anything else is dropped and printed.

It deliberately does NOT use plausible() to break the tie, though the
cross-printing split does. plausible() does not recognise the Fairchild 93xx and
96xx series: it calls 9312, 9322 and 9602 implausible, and 9316 too — which this
repo's own equivalence table documents as Fairchild's 74161. Filtering on it here
would have discarded the 9312 reading of Indy 4's B3 and "resolved" that cell to
a 7474, a different device entirely. A false correction is worse than the
collision it replaces. The split path has the same blind spot and is now flagged
in HANDOFF, unaudited.

The fix also unblocks the two boards withheld last time for exactly this reason.
Pole Position II (38 devices, 8 cells dropped) and Xevious (18, 1 dropped) no
longer need figure-splitting to be safe, because a cell nothing can attribute is
now simply absent rather than guessed.

47 boards, 2,489 devices.

Co-Authored-By: Claude Opus 5 <noreply@anthropic.com>
Parts:
- removed U10B: 74S00, DIP-14_W7.62mm
- removed U1A: 74LS157, DIP-16_W7.62mm
- removed U1B: 74LS244, DIP-20_W7.62mm
- removed U2H, U9B: 74LS374, DIP-20_W7.62mm
- removed U3H: 74LS257, DIP-16_W7.62mm
- removed U4P: 74LS27, DIP-14_W7.62mm
- removed U7L: 74S08, DIP-14_W7.62mm

Commit message: Split two maps that were two PCBs stacked
The collision work catches a manual whose PCBs share designators: C1 on one is
not C1 on the other, the cell is claimed twice, something notices. It cannot
catch the quieter case. Two PCBs whose designators do not overlap merge into a
single map with no collision, no warning, and a result that looks complete.

Asking of every published board whether its trusted rows sat under more than one
figure heading naming a different PCB found two: I, Robot (an I, ROBOT CPU PCB
and an I, ROBOT Video PCB) and Paperboy (a Central Processing Unit PCB and a
Video PCB). Both published one map covering both boards. That is worse than an
incomplete map — a repairer reading cell 5A off it is being told something
false, because 5A exists on both boards and means different things.

Split. The existing slug keeps the CPU board, so its URL and anything pointing
at it stay valid, and the video board is new. Splitting recovers devices rather
than losing them — I, Robot goes from 45 to 33 plus 24 — because cells both
boards claimed had been dropped as collisions and are separable once the boards
are.

Three more took a handful of devices from the wrong board's figure: Tempest 5
from its Auxiliary PCB on a map that is the Analog Vector-Generator PCB, Pole
Position 4 sitting under a video-display monitor list as readily as the CPU one,
Food Fight 1 shared with an EMI Shield figure. Removed and re-harvested under
each board's own figure, where all three add nothing back — which is what
confirms the five, four and one were never theirs.

Millipede looked identical and is not. Its TM-217 has one figure heading the
regex recognises, so all 46 rows inherit 'Utility Panel Assembly' — but they are
game-PCB TTL and a utility panel does not carry 46 logic chips. Meaningless
attribution rather than a wrong board, and its two printings agree. Left alone.

Splitting also exposed that merge_ic_locations keeps lookup entries not on the
grid, by design, for crystals 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
Parts:
- removed U10A, U5K, U5L: 74S157, DIP-16_W7.62mm
- removed U12E: 74153, DIP-16_W7.62mm
- removed U12P: 74S00, DIP-14_W7.62mm
- removed U13K, U13L: 74LS174, DIP-16_W7.62mm
- removed U2L: 74LS157, DIP-16_W7.62mm
- removed U3B: 74LS08, DIP-14_W7.62mm
- removed U3L: 74LS257, DIP-16_W7.62mm
- removed U5R: 74S04, DIP-14_W7.62mm
- removed U8M: 74LS04, DIP-14_W7.62mm
- removed U8N: 74LS00, DIP-14_W7.62mm
- removed U8P: 74LS74, DIP-14_W7.62mm
- removed U8R: 74S08, DIP-14_W7.62mm
- removed U9A: 74LS374, DIP-20_W7.62mm
- removed U9C, U9D: 74LS85, DIP-16_W7.62mm
- added U10B: 74S32, DIP-14_W7.62mm, F.Cu at (254.6, 227.6)
- added U1B: 74LS32, DIP-14_W7.62mm, F.Cu at (26.0, 227.6)
- added U2H: 74LS245, DIP-20_W7.62mm, F.Cu at (51.4, 132.3)
- added U3H: 74LS244, DIP-20_W7.62mm, F.Cu at (76.8, 132.3)
- added U7L: 74S163, DIP-16_W7.62mm, F.Cu at (178.4, 94.2)
- added U9B: 74LS00, DIP-14_W7.62mm, F.Cu at (229.2, 227.6)
