File: kicad/i-robot-video/i-robot-video.kicad_pcb (KiCad board)
At the start: 2 copper layers, 315 x 257 mm, 27 parts, among them U10C 7406, U10M 74LS161, U10N 74LS161, U1F 74LS86, U1H 7407, U2C 74S08, U2D 74S157, U2H 74LS74, U2K 74LS74, U3B 74LS157, U3P 74LS157, U4C 74LS86, U4F 74LS273, U4K 74LS367, U4L 74LS157, U4M 74LS157, U4N 74LS157, U4P 74S00, U5M 74LS194, U5N 74LS194, U6B 74LS273, U6H 74LS157, U6K 74LS273, U7M 74LS273, U8H 74LS245, U8M 74LS244, U8N 74LS244

Commit message: Split two maps that were two PCBs stacked
The collision work catches a manual whose PCBs share designators: C1 on one is
not C1 on the other, the cell is claimed twice, something notices. It cannot
catch the quieter case. Two PCBs whose designators do not overlap merge into a
single map with no collision, no warning, and a result that looks complete.

Asking of every published board whether its trusted rows sat under more than one
figure heading naming a different PCB found two: I, Robot (an I, ROBOT CPU PCB
and an I, ROBOT Video PCB) and Paperboy (a Central Processing Unit PCB and a
Video PCB). Both published one map covering both boards. That is worse than an
incomplete map — a repairer reading cell 5A off it is being told something
false, because 5A exists on both boards and means different things.

Split. The existing slug keeps the CPU board, so its URL and anything pointing
at it stay valid, and the video board is new. Splitting recovers devices rather
than losing them — I, Robot goes from 45 to 33 plus 24 — because cells both
boards claimed had been dropped as collisions and are separable once the boards
are.

Three more took a handful of devices from the wrong board's figure: Tempest 5
from its Auxiliary PCB on a map that is the Analog Vector-Generator PCB, Pole
Position 4 sitting under a video-display monitor list as readily as the CPU one,
Food Fight 1 shared with an EMI Shield figure. Removed and re-harvested under
each board's own figure, where all three add nothing back — which is what
confirms the five, four and one were never theirs.

Millipede looked identical and is not. Its TM-217 has one figure heading the
regex recognises, so all 46 rows inherit 'Utility Panel Assembly' — but they are
game-PCB TTL and a utility panel does not carry 46 logic chips. Meaningless
attribution rather than a wrong board, and its two printings agree. Left alone.

Splitting also exposed that merge_ic_locations keeps lookup entries not on the
grid, by design, for crystals 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
Parts:
- removed U10C: 7406, DIP-14_W7.62mm
- removed U10M, U10N: 74LS161, DIP-16_W7.62mm
- removed U1F, U4C: 74LS86, DIP-14_W7.62mm
- removed U1H: 7407, DIP-14_W7.62mm
- removed U2C: 74S08, DIP-14_W7.62mm
- removed U2D: 74S157, DIP-16_W7.62mm
- removed the U2H at (51.4, 113.2)
- removed U2K: 74LS74, DIP-14_W7.62mm
- removed the U3B at (76.8, 208.5)
- removed U3P, U4L, U4M, U4N, U6H: 74LS157, DIP-16_W7.62mm
- removed U4F, U6B, U6K, U7M: 74LS273, DIP-20_W7.62mm
- removed U4K: 74LS367, DIP-16_W7.62mm
- removed U5M, U5N: 74LS194, DIP-16_W7.62mm
- removed U8H: 74LS245, DIP-20_W7.62mm
- removed the U8M at (203.8, 56.1)
- removed the U8N at (203.8, 27.5)
- added U10A: 74S157, DIP-16_W7.62mm, F.Cu at (254.6, 246.6)
- added U12E: 74153, DIP-16_W7.62mm, F.Cu at (305.4, 170.4)
- added U12P: 74S00, DIP-14_W7.62mm, F.Cu at (305.4, 37.0)
- added U13K: 74LS174, DIP-16_W7.62mm, F.Cu at (330.8, 113.2)
- added U13L: 74LS174, DIP-16_W7.62mm, F.Cu at (330.8, 94.2)
- added U1B: 74LS244, DIP-20_W7.62mm, F.Cu at (26.0, 227.6)
- added U2H: 74LS374, DIP-20_W7.62mm, F.Cu at (51.4, 132.3)
- added U2L: 74LS157, DIP-16_W7.62mm, F.Cu at (51.4, 94.2)
- added U3B: 74LS08, DIP-14_W7.62mm, F.Cu at (76.8, 227.6)
- added U3H: 74LS257, DIP-16_W7.62mm, F.Cu at (76.8, 132.3)
- added U3L: 74LS257, DIP-16_W7.62mm, F.Cu at (76.8, 94.2)
- added U5K: 74S157, DIP-16_W7.62mm, F.Cu at (127.6, 113.2)
- added U5L: 74S157, DIP-16_W7.62mm, F.Cu at (127.6, 94.2)
- added U5R: 74S04, DIP-14_W7.62mm, F.Cu at (127.6, 18.0)
- added U7L: 74S08, DIP-14_W7.62mm, F.Cu at (178.4, 94.2)
- added U8M: 74LS04, DIP-14_W7.62mm, F.Cu at (203.8, 75.2)
- added U8N: 74LS00, DIP-14_W7.62mm, F.Cu at (203.8, 56.1)
- added U8P: 74LS74, DIP-14_W7.62mm, F.Cu at (203.8, 37.0)
- added U8R: 74S08, DIP-14_W7.62mm, F.Cu at (203.8, 18.0)
- added U9A: 74LS374, DIP-20_W7.62mm, F.Cu at (229.2, 246.6)
- added U9B: 74LS374, DIP-20_W7.62mm, F.Cu at (229.2, 227.6)
- added U9C: 74LS85, DIP-16_W7.62mm, F.Cu at (229.2, 208.5)
- added U9D: 74LS85, DIP-16_W7.62mm, F.Cu at (229.2, 189.4)
- U4P: value 74S00 -> 74LS27
- moved U4P 19.0 mm to (102.2, 37.0)
Other:
- board size 315 x 257 mm -> 544 x 276 mm
