File: kicad/paperboy/paperboy.kicad_pcb (KiCad board)
At the start: 2 copper layers, 315 x 276 mm, 20 parts, among them U11D 74S08, U1C 74LS157, U1K 74LS245, U2F 74LS244, U2M 74LS139, U2N 74LS374, U4A 74LS244, U4F 74LS393, U5A 74S04, U5B 74LS109, U5J 74LS08, U5K 74LS04, U5L 74LS139, U5N 74LS174, U5P 74LS244, U6D 74LS245, U7H 74LS74, U7R 74LS161, U8B 74LS161, U8N 74S04

Commit message: Split two maps that were two PCBs stacked
The collision work catches a manual whose PCBs share designators: C1 on one is
not C1 on the other, the cell is claimed twice, something notices. It cannot
catch the quieter case. Two PCBs whose designators do not overlap merge into a
single map with no collision, no warning, and a result that looks complete.

Asking of every published board whether its trusted rows sat under more than one
figure heading naming a different PCB found two: I, Robot (an I, ROBOT CPU PCB
and an I, ROBOT Video PCB) and Paperboy (a Central Processing Unit PCB and a
Video PCB). Both published one map covering both boards. That is worse than an
incomplete map — a repairer reading cell 5A off it is being told something
false, because 5A exists on both boards and means different things.

Split. The existing slug keeps the CPU board, so its URL and anything pointing
at it stay valid, and the video board is new. Splitting recovers devices rather
than losing them — I, Robot goes from 45 to 33 plus 24 — because cells both
boards claimed had been dropped as collisions and are separable once the boards
are.

Three more took a handful of devices from the wrong board's figure: Tempest 5
from its Auxiliary PCB on a map that is the Analog Vector-Generator PCB, Pole
Position 4 sitting under a video-display monitor list as readily as the CPU one,
Food Fight 1 shared with an EMI Shield figure. Removed and re-harvested under
each board's own figure, where all three add nothing back — which is what
confirms the five, four and one were never theirs.

Millipede looked identical and is not. Its TM-217 has one figure heading the
regex recognises, so all 46 rows inherit 'Utility Panel Assembly' — but they are
game-PCB TTL and a utility panel does not carry 46 logic chips. Meaningless
attribution rather than a wrong board, and its two printings agree. Left alone.

Splitting also exposed that merge_ic_locations keeps lookup entries not on the
grid, by design, for crystals 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
Parts:
- removed U11D: 74S08, DIP-14_W7.62mm
- removed U1C: 74LS157, DIP-16_W7.62mm
- removed U2M: 74LS139, DIP-16_W7.62mm
- removed U2N: 74LS374, DIP-20_W7.62mm
- removed U5A: 74S04, DIP-14_W7.62mm
- removed U5B: 74LS109, DIP-16_W7.62mm
