File: kicad/pole-position/pole-position.kicad_pcb (KiCad board)
At the start: 2 copper layers, 366 x 257 mm, 49 parts, among them U10B 74LS74, U10D 74LS174, U10E 74LS257, U10N 74LS85, U11B 74107, U11C 7497, U11F 74LS174, U11H 74LS174, U11K 74LS139, U12C 74LS161, U12D 74LS393, U12F 74LS86, U13F 74LS20, U1B 74107, U2E 74LS74, U2H 74LS139, U3H 74LS175, U4B 74LS367, U4C 74LS373, U4H 74LS157, U4K 74LS174, U4M 74LS373, U5A 74LS74, U5B 74LS174, U5C 74LS174, U5F 74LS245, U5H 74LS175, U5K 74LS244, U5N 74LS74, U6H 74LS245, U6L 74LS109, U7C 74S04, U7D 74LS32, U7L 74LS273, U7M 74LS273, U7N 74S04, U8B 74S00, U8C 74LS157, U8E 74LS259, U8F 74LS367, U8K 4066, U8M 74LS04, U9B 74LS20, U9C 74LS157, U9E 74LS257, U9H 74LS161, U9K 7497, U9L 74LS174, U9N 74LS85

Commit message: Teach plausible() the Fairchild parts; audit what it had decided
The last commit flagged that plausible() does not recognise the Fairchild
93xx/96xx series and left it unaudited. Audited now.

plausible() called 9312, 9316, 9321, 9322, 9300, 9301, 9334 and 9602
implausible — eight parts in 111 trusted rows and on 64 devices of published
maps, every one of them admitted by well_formed(). The two functions disagreed
about real parts, and 9316 is one this repo's own equivalence table documents
as Fairchild's 74161. Bounded to 9[36]\d{2}: a bare 9\d{3} would admit any
four-digit OCR smear.

The audit replayed the cross-printing split over every published board. 8 cells
had been decided by the filter. 4 were Asteroids P9, where a printing reading
9316 lost to one reading 74LS164 — the blind spot, discarding the more specific
reading as wreckage — and P9 is on none of the four Asteroids maps. The other 4
were the filter doing its job: 8728 to 8T28 on Football, 74LSI91 to 74LS191 on
Major Havoc, capital-I read as 1. After the fix 4 remain, all of the second
kind. No published device ever came from a false resolution.

Dropping a contested cell frees the readings a collision used to consume, so a
re-merge recovers 9 devices: Monte Carlo 3, Pole Position 4, Food Fight 1,
Soccer 1. Checked first that none of the 22 cells withdrawn last commit would
come back — every one is still reported as contested.

APB exposed a separate fault. Its 3B/F span names rows five apart, build_board
raised on it, and removing it by hand did not stick because the next merge wrote
it again — the adjacency rule lived only at build time, after the board file was
already wrong. It now runs where the designator is first accepted, and says so:
"impossible span 3B/F — those rows are not adjacent on this grid".

All 47 boards build. 2,498 devices.

Co-Authored-By: Claude Opus 5 <noreply@anthropic.com>
Parts:
- added U10H: 74LS273, DIP-20_W7.62mm, F.Cu at (254.6, 113.2)
- added U10K: 4066, DIP-14_W7.62mm, F.Cu at (254.6, 75.2)
- added U10L: 4066, DIP-14_W7.62mm, F.Cu at (254.6, 56.1)
- added U6C: 74LS08, DIP-14_W7.62mm, F.Cu at (153.0, 189.4)

Commit message: Split two maps that were two PCBs stacked
The collision work catches a manual whose PCBs share designators: C1 on one is
not C1 on the other, the cell is claimed twice, something notices. It cannot
catch the quieter case. Two PCBs whose designators do not overlap merge into a
single map with no collision, no warning, and a result that looks complete.

Asking of every published board whether its trusted rows sat under more than one
figure heading naming a different PCB found two: I, Robot (an I, ROBOT CPU PCB
and an I, ROBOT Video PCB) and Paperboy (a Central Processing Unit PCB and a
Video PCB). Both published one map covering both boards. That is worse than an
incomplete map — a repairer reading cell 5A off it is being told something
false, because 5A exists on both boards and means different things.

Split. The existing slug keeps the CPU board, so its URL and anything pointing
at it stay valid, and the video board is new. Splitting recovers devices rather
than losing them — I, Robot goes from 45 to 33 plus 24 — because cells both
boards claimed had been dropped as collisions and are separable once the boards
are.

Three more took a handful of devices from the wrong board's figure: Tempest 5
from its Auxiliary PCB on a map that is the Analog Vector-Generator PCB, Pole
Position 4 sitting under a video-display monitor list as readily as the CPU one,
Food Fight 1 shared with an EMI Shield figure. Removed and re-harvested under
each board's own figure, where all three add nothing back — which is what
confirms the five, four and one were never theirs.

Millipede looked identical and is not. Its TM-217 has one figure heading the
regex recognises, so all 46 rows inherit 'Utility Panel Assembly' — but they are
game-PCB TTL and a utility panel does not carry 46 logic chips. Meaningless
attribution rather than a wrong board, and its two printings agree. Left alone.

Splitting also exposed that merge_ic_locations keeps lookup entries not on the
grid, by design, for crystals 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
Parts:
- removed U10H: 74LS273, DIP-20_W7.62mm
- removed U10K, U10L: 4066, DIP-14_W7.62mm
- removed U6C: 74LS08, DIP-14_W7.62mm
