File: kicad/asteroids-05/asteroids-05.kicad_pcb (KiCad board)
At the start: 2 copper layers, 300 x 330 mm, 100 parts

Commit message: Draw every device at its real package size
The board maps existed to answer "which chip is at C4", and then drew a
24-pin ROM and a 20-pin LS245 as the same 14-pin outline. package_for()
read pin counts from DEVICES, which holds 20 Pong-era parts against the
112 part types the boards actually use, and silently fell back to DIP-14
for the other 92.

tools/packages.py is the pin-count table, kept separate from devices.py
on purpose: packaging needs one number for every part on every board,
while devices.py carries verified pinouts for the parts validate_nets.py
reasons about, and widening that set to satisfy a drawing would let the
extractor trust readings nothing has checked.

688 of 704 devices now size. check_packages.py re-derives 56 of the
entries from KiCAD's symbol library — comparing the highest pin number,
not the pin count, since KiCAD omits no-connects and a 7493 symbol has
ten pins on a DIP-14 — and confirms all 20 parts in DEVICES agree. The
Am2901 slices and the POKEY come from DIP-40 stated on the Battlezone
sheet; the 8316E from the drawing's note that a 2708 may be fitted
instead.

What does not size is now said out loud rather than quietly drawn at 14
pins: four descriptions recorded where the sheet gave no part number,
and the Atari 0351xx ROM/PROM numbers, which get the class default and
are listed as unverified until someone has a board in front of them.

Two things found while reading the corpus for packages, both logged in
asteroids.read.json rather than acted on. The -06 rate multiplier
resolution was recorded and never applied to the board data, and the
parts list disagrees with both readings on designators. F4/H4/J4 take
either an LS670 or an LS170, and the 19-007 pull-up network is fitted
only with the LS170 — same package either way, but a real failure mode.

Also: republishing a board without --machine used to unlink it from its
machine, because most definitions carry no machine of their own and the
link lived only in boards.json. publish_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
Parts:
- UA10, UB12, UB7, UC10, UC11, UC7, UC8, UD10, UD12, UD7, UD9, UE10, UE11, UE7, UF10, UF11, UF3, UF4, UF5, UF6, UF9, UH10, UH3, UH4, UH5, UH6, UH9, UJ10, UJ11, UJ3, UJ4, UJ5, UJ6, UJ9, UK3, UK5, UK9, UL11, UL3, UM11, UM6, UM7, UN11: footprint DIP-14_W7.62mm -> DIP-16_W7.62mm
- UB16, UB2, UC2, UE3, UF7, UH7, UJ7, UK7, UR2: footprint DIP-14_W7.62mm -> DIP-20_W7.62mm
- UC3: footprint DIP-14_W7.62mm -> DIP-40_W15.24mm
- UD2, UE2, UK4, UL4, UM4, UN4, UP4, UR4: footprint DIP-14_W7.62mm -> DIP-18_W7.62mm
- UF2, UH2, UJ2, UM2, UN2, UN3: footprint DIP-14_W7.62mm -> DIP-24_W15.24mm
- UL10, UM9: footprint DIP-14_W7.62mm -> DIP-8_W7.62mm

Commit message: Drop two grid rows that do not exist, and span the devices that do
Atari's grid alphabet skips G, I, O and Q, and the board definitions
listed G and Q as rows. Every device below F was therefore drawn a row
too low, the rendered board carried two empty bands, and F/H1 looked
like a three-position span for a part 1.2in long on a 0.75in pitch.

Confirmed three ways before touching it. Nothing in any read, signature
or signal record in this repo sits in a G or Q row, while both
neighbours of each are populated on the two densest boards — Battlezone
P:6 R:2, Asteroids-03 P:4 R:3. The sheets' own spanning designators
treat F and H as adjacent and H and J as adjacent, which is only
possible if G and I are not positions. And with G removed, F/H falls out
as an adjacent pair, which is what a 24-pin ROM needs. Pong predates the
convention and legitimately uses G, so it keeps its grid.

Spans are now data rather than prose. A device drawn across two or three
cells is still keyed at its first cell, because that is the only thing
`ics` may be keyed by, but the sheet's own designator goes in a `spans`
map and the footprint is placed at the mean of the cells it names. A
DIP-40 at B/C2 sits between B2 and C2 instead of hanging equally over A2
and C2. The build rejects a span whose rows are not adjacent — that
failure almost always means the grid is wrong, not the span.

Two more inconsistencies found and logged rather than guessed at. Two of
the Math Box's four Am2901 slices carry a span and two do not, though
all four are the same DIP-40 on the same pitch. And asteroids-04.json
carries five devices at the -03 PROM positions alongside the -04 ROMs
and is missing 035144-02 at D/E1, contradicting the substitution table,
memory_by_revision and its own status text in the same breath.

Co-Authored-By: Claude Opus 5 <noreply@anthropic.com>
Parts:
- moved UA10 38.1 mm to (254.6, 265.6)
- moved UA7 38.1 mm to (178.4, 265.6)
- moved UA9 38.1 mm to (229.2, 265.6)
- moved UE10 38.1 mm to (254.6, 189.4)
- moved UE11 38.1 mm to (280.0, 189.4)
- moved UE12 38.1 mm to (305.4, 189.4)
- moved UE2 38.1 mm to (51.4, 189.4)
- moved UE3 38.1 mm to (76.8, 189.4)
- moved UE5 38.1 mm to (127.6, 189.4)
- moved UE6 38.1 mm to (153.0, 189.4)
- moved UE7 38.1 mm to (178.4, 189.4)
- moved UB12 38.1 mm to (305.4, 246.6)
- moved UB16 38.1 mm to (407.0, 246.6)
- moved UB2 38.1 mm to (51.4, 246.6)
- moved UB4 38.1 mm to (102.2, 246.6)
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
Commit message: Fix the Asteroids revision complements at their source
build_asteroids_revisions.py overlaid each revision's memory onto the
base sheet read without clearing what that memory replaces, so -04, -05
and -06 all carried leftover -03 PROM positions — a -04 board map
claiming five PROMs the -04 does not have, next to its own status text
saying three ROMs replace all eleven. Its grid filter also dropped any
designator containing a slash, which is why each revision was missing
exactly one of its own ROMs: 035144-02 at D/E1 on the -04, 035143-02 at
E/F2 on the -05 and -06. All four revisions now match the substitution
table exactly, and the spanning ROMs are placed across both cells.

The generator emits data/chips/<slug>.json too. That file is what the
site's "which chip is at C4" lookup reads, nothing generated it, and it
had drifted from the board maps in the obvious way — showing the sheet's
'ROM 035131' at J2 where the map showed the table's '035131-02', and
still listing the leftovers. Twenty-three entries change and every one
is accounted for.

It now reports collisions rather than letting dict ordering settle them,
which surfaced three that were being decided silently. B10's alternate
is recorded as B9 and is the only one of twenty-eight that shifts down;
it collides with B8's, so a -05/-06 board has two devices claiming B9.
D12 reads as a 74LS374 on sheet 02A and a CD4016B on 02B. E2 on -05/-06
is the sheet's 2114 against the table's 035143-02 at E/F2. The table
wins that one, being typeset and revision-specific; the other two are
logged, because B10->B11 is a pattern I can see and not a reading.

The -05/-06 status text claimed a designator shift. The drawing gives
the alternate for only 28 of the 106 devices read, so the other 78 sit
at their -03/-04 positions and the text now says that.

Co-Authored-By: Claude Opus 5 <noreply@anthropic.com>
Parts:
- removed UF2: ROM 035135, DIP-24_W15.24mm
- removed UM2: ROM 035134, DIP-24_W15.24mm
- removed UN2: ROM 035132, DIP-24_W15.24mm
- UE2: value 2114 -> 035143-02; footprint DIP-18_W7.62mm -> DIP-24_W15.24mm
- moved UE2 9.52 mm to (51.4, 179.9)

Commit message: Name the four parts the sheets never did
C5, E12 and M12 on Asteroids were recorded by function — "counter",
"op-amp", "DIP switch" — because the drawings give no part number for
them, and they were the last devices the board maps could not size. The
parts lists give all three, and agree across printings.

C5 is a 9316. Five printings name a counter there: the 6th, 7th and
Cocktail 3rd say 37-9316, the 1st and 2nd say 37-74LS161, and the 9316
is Fairchild's 74161, so those are the same part and not a conflict. It
matches the read's own note that C5 divides 3kHz by 12 for the NMI.

E12 is Atari 137108-001, item 130, "Operational Amplifier Integrated
Circuit", at E12 in three printings; the Caberat manual names the type,
TL081CP. Same designator, same block, three documents. The same item
also lists a B/C12 location that nothing in the read accounts for, which
is noted and not acted on.

M12 is Atari 66-114P1T, a 4-station DIP switch, item 143 at M12 in three
printings. Sized as DIP-8, since n SPST switches in a DIP is 2n pins;
the 8-station switches on Battlezone and Tempest are DIP-16 for the same
reason.

All three are cross-document confirmations rather than re-readings of
the same sheet, which is the route the house rules say to try first and
the one that has resolved every conflict here so far. Every device on
every board now has a package: 106 of 106 part types, 694 of 694
devices. What remains unverified is the twenty Atari 0351xx ROM/PROM
positions, drawn on a class default, and those want a board.

Co-Authored-By: Claude Opus 5 <noreply@anthropic.com>
Parts:
- UC5: value counter -> 9316; footprint DIP-14_W7.62mm -> DIP-16_W7.62mm
- UE12: value op-amp -> 137108-001; footprint DIP-14_W7.62mm -> DIP-8_W7.62mm
- UM12: value DIP switch -> 4-position DIP switch; footprint DIP-14_W7.62mm -> DIP-8_W7.62mm

Commit message: Settle four gaps from outside sources, and find a fifth inside
Researching the open questions turned up a source that was in the corpus
all along. Atari stocked IC sockets by contact count, so a parts list
row like '79-42C24 24-Contact Medium-Insertion-Force Integrated Circuit
Socket (J2, H2, E/F2, N/P3)' states the pin count of every socketed
position, in the same typeset list the devices come from.
check_socket_pins.py checks packages.py against it: 26 sizes confirmed,
none contradicted. It needs the same --docs and --figure targeting the
merge does — pooled by machine it mixes Battlezone's two PCBs and
compares one printing's numbering against another's, and reported
thirteen contradictions that were all artefacts of that.

The Atari ROM sizes are no longer a class default. Those sockets are the
program ROM and vector ROM positions, and they are 24-contact.

The -05/-06 ROM positions were the wrong way round. 035143-02 is at J2
and 035145-02 at E/F2, not the reverse. Three sources agree and two are
in this corpus: the 6th and 7th printings both list the positions
outright, and MAME's asteroid driver names its dumps 035143-02.j2 and
035145-04e.ef2, its suffixes being board positions checked against real
boards. 035144-02 at H2 was right all along; only the outer two were
swapped.

The twelfth -03 PROM is real and is in — 035142-02 at L1, with 035155-02
as its alternate. Sheet 01B of the 4th-printing drawing package carries
'035142-01 L1' directly, which is the drawing rather than a manual
quoting it, six further documents repeat it, and the memory map requires
it: 6800-7FFF is 6144 bytes, exactly twelve 512-byte PROMs or three 2K
ROMs and nothing else that tiles evenly. Eleven could never have been
right.

Missile Command D3 is a 74LS14 and the 7404 reading is withdrawn. All
five printings give '37-74LS14 Type 74LS14 Integrated Circuit (D3)' with
stock number and description agreeing in each, and the same rows put a
plain 7414 at J9, so the lists distinguish the t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
Parts:
- UE2: value 035143-02 -> 035145-02
- UJ2: value 035145-02 -> 035143-02

Commit message: Put MAME's ROM positions on the maps; let the late Asteroids boards take the lists
Two things declined earlier as decisions rather than chores, reconsidered.

The parts-list harvest never reaches memory. Atari stocks ROMs and PROMs under
its own part numbers, not as 37-series IC stock, so those rows fail the
checksum the harvest depends on — which is why Red Baron's whole complement was
missing once, and why 79 memory cells on 15 boards sat empty with everything
around them filled. MAME has them: its ROM file names encode the board
position — 035224.e2 is part 035224 at E2, 037587-01.fh1 is at the span F/H1 —
and they were checked against real boards by the people who dumped them. The
site already publishes those maps as their own asset with their own caveat.
This is that source reaching the board map under the same label, not a new one
mixed in quietly: 78 devices on 14 boards, each recorded in the chip lookup as
"MAME ROM map", only where the map had nothing. The three cells where a parts
list and MAME disagree are untouched and stay logged.

Asteroids -05 and -06 were left without the parts lists because those are
written in early designators and a direct merge would put a device one column
from where the board has it. So they take -03's parts-list additions instead,
shifted through the drawing's early-to-late table where an alternate is known
and placed at the early cell otherwise — which is exactly what these boards
already do for their 78 unshifted drawing-read devices, under a caveat they
already carry. 13 each. None of the 22 turned out to have a known alternate,
and 9 land on cells a shifted device already occupies and are skipped rather
than duplicated. All of it runs inside the generator, so it survives
regeneration.

50 boards, 2,672 devices.

Co-Authored-By: Claude Fable 5.1 <noreply@anthropic.com>
Parts:
- added UA11: 74LS157, DIP-16_W7.62mm, F.Cu at (280.0, 265.6)
- added UB13: 4016B, DIP-14_W7.62mm, F.Cu at (330.8, 246.6)
- added UE4: 74LS139, DIP-16_W7.62mm, F.Cu at (102.2, 189.4)
- added UE8: 74LS42, DIP-16_W7.62mm, F.Cu at (203.8, 189.4)
- added UN12: 74LS174, DIP-16_W7.62mm, F.Cu at (305.4, 56.1)
- added UN7: 74LS174, DIP-16_W7.62mm, F.Cu at (178.4, 56.1)
- added UP2: 74LS245, DIP-20_W7.62mm, F.Cu at (51.4, 37.0)
- added UP6: 74LS253, DIP-16_W7.62mm, F.Cu at (153.0, 37.0)
- added UP7: 74LS174, DIP-16_W7.62mm, F.Cu at (178.4, 37.0)
- added UP8: 74LS161, DIP-16_W7.62mm, F.Cu at (203.8, 37.0)
- added UR11: 4016B, DIP-14_W7.62mm, F.Cu at (280.0, 18.0)
- added UR12: 4016B, DIP-14_W7.62mm, F.Cu at (305.4, 18.0)
- added UR7: 74LS08, DIP-14_W7.62mm, F.Cu at (178.4, 18.0)
