File: kicad/battlezone/battlezone.kicad_pcb (KiCad board)
At the start: 2 copper layers, 300 x 300 mm, 23 parts

Commit message: Deepen the Centipede and Battlezone board maps
Centipede gains sheet 02A: the playfield address selector and the eight
2101A-2 playfield RAMs, taking it from 13 devices to 23. The sheet also carries
a complete playfield RAM test — CAT Box switch settings, key in 0400, and a lit
COMPARE ERROR LED gives the failing address directly.

Battlezone gains sheet 02B: both 8-position option switch banks (M10 read by
N11 via OPT0, P10 read by P11 via OPT1), the coin door input buffer and the
Y-axis DAC. 23 devices to 31.

Worth knowing from that sheet: R11 buffers the coin door inputs *and* 3KHZ and
HALT, so a machine that will not coin up and one reporting a bad
vector-generator state can share a single failed buffer.

Adds tools/publish_board.py — interactive view, BOM and site registration in
one command, rather than three ad-hoc snippets per board.

Co-Authored-By: Claude Opus 5 <noreply@anthropic.com>
Parts:
- added UC8: 74LS273, DIP-14_W7.62mm, F.Cu at (203.8, 265.6)
- added UC9: DAC-08, DIP-14_W7.62mm, F.Cu at (229.2, 265.6)
- added UM10: 8-position DIP switch, DIP-14_W7.62mm, F.Cu at (254.6, 94.2)
- added UN11: 74LS244, DIP-14_W7.62mm, F.Cu at (280.0, 75.2)
- added UP10: 8-position DIP switch, DIP-14_W7.62mm, F.Cu at (254.6, 56.1)
- added UP11: 74LS244, DIP-14_W7.62mm, F.Cu at (280.0, 56.1)
- added UR11: 74LS244, DIP-14_W7.62mm, F.Cu at (280.0, 18.0)
- added UR9: 74S04, DIP-14_W7.62mm, F.Cu at (229.2, 18.0)

Commit message: Read Battlezone sheet 3, the whole digital vector generator
Sheet 2 was the only Battlezone sheet read, and it was read thinly: 31
devices, with program memory, power regulation, the NMI counter and half
the address decoder untouched. Sheet 3 Side A was untouched entirely.

Both are now read by eye, block by block, taking the board from 31 devices
to 97. Sheet 3 is the vector generator end to end -- stack and program
counter, address selector, vector RAM and ROM, data buffer and shifter,
state machine, vector timer and the halt latch.

Two findings that change how the board reads:

The vector state PROM is K7, an 82S129 carrying Atari 036408, with L7 as
the state register and J7 decoding STATE0-2 into the strobes and latches.
A vector generator stuck in one state is those three chips. HALT is
latched at M9 and cleared by VGGO, and it is the same HALT the coin-door
buffer R11 reads back on sheet 2 -- so the self-test indication and the
generator's own halt are one signal, not two.

Sheets 2 and 3 are sections of the same 035742 PCB, so they share one
designator grid, and eight packages appear on both sheets using different
halves: C4, L10, M7, J4, K4, B6, R9 and K2. Every one of them read as the
same part on both sheets, which is the strongest cross-check available
without a physical board.

Logged rather than guessed: R9, R10 and R11 are ICs at those grid
positions on sheets 2B and 3A, and also ordinary resistor numbers on
sheets 2A and 3A. Nothing distinguishes them but the symbol they are
drawn as. That is not fixable by renaming -- it has to be read off the
drawing every time.

Corrected: the LS245 alternate is AM8304B, not AM83048, confirmed on both
sheets; and sheet 2 has two of them, P4 and P2, where only P4 was
recorded. The MPU's own designator is L/M/N3, spanning three grid cells,
the same convention as the L/M1 and F/H1 ROMs.

Co-Authored-By: Claude Opus 5 <noreply@anthropic.com>
Parts:
- added UA1: 2114, DIP-14_W7.62mm, F.Cu at (26.0, 303.8)
- added UA2: 2114, DIP-14_W7.62mm, F.Cu at (51.4, 303.8)
- added UA3: 8316E, DIP-14_W7.62mm, F.Cu at (76.8, 303.8)
- added UA5: 74LS194, DIP-14_W7.62mm, F.Cu at (127.6, 303.8)
- added UA6: 74LS194, DIP-14_W7.62mm, F.Cu at (153.0, 303.8)
- added UB1: 2114, DIP-14_W7.62mm, F.Cu at (26.0, 284.7)
- added UB2: 2114, DIP-14_W7.62mm, F.Cu at (51.4, 284.7)
- added UB3: 8316E, DIP-14_W7.62mm, F.Cu at (76.8, 284.7)
- added UB4: 74LS42, DIP-14_W7.62mm, F.Cu at (102.2, 284.7)
- added UB5: 74LS194, DIP-14_W7.62mm, F.Cu at (127.6, 284.7)
- added UB7: 74S86, DIP-14_W7.62mm, F.Cu at (178.4, 284.7)
- added UC1: 2114, DIP-14_W7.62mm, F.Cu at (26.0, 265.6)
- added UC2: 2114, DIP-14_W7.62mm, F.Cu at (51.4, 265.6)
- added UC5: 74LS194, DIP-14_W7.62mm, F.Cu at (127.6, 265.6)
- added UC6: 74S00, DIP-14_W7.62mm, F.Cu at (153.0, 265.6)
- added UD1: 2114, DIP-14_W7.62mm, F.Cu at (26.0, 246.6)
- added UD2: 2114, DIP-14_W7.62mm, F.Cu at (51.4, 246.6)
- added UD4: 74LS157, DIP-14_W7.62mm, F.Cu at (102.2, 246.6)
- added UD5: 74LS194, DIP-14_W7.62mm, F.Cu at (127.6, 246.6)
- added UD6: 74LS194, DIP-14_W7.62mm, F.Cu at (153.0, 246.6)
- added UE1: 8316E, DIP-14_W7.62mm, F.Cu at (26.0, 227.6)
- added UE3: 8316E, DIP-14_W7.62mm, F.Cu at (76.8, 227.6)
- added UE4: 74LS157, DIP-14_W7.62mm, F.Cu at (102.2, 227.6)
- added UE5: 74LS193, DIP-14_W7.62mm, F.Cu at (127.6, 227.6)
- added UE6: 74LS670, DIP-14_W7.62mm, F.Cu at (153.0, 227.6)
- added UF1: 8316E, DIP-14_W7.62mm, F.Cu at (26.0, 208.5)
- added UF10: 74LS191, DIP-14_W7.62mm, F.Cu at (254.6, 208.5)
- added UF2: 74LS245, DIP-14_W7.62mm, F.Cu at (51.4, 208.5)
- added UF3: 8316E, DIP-14_W7.62mm, F.Cu at (76.8, 208.5)
- added UF4: 74LS157, DIP-14_W7.62mm, F.Cu at (102.2, 208.5)
- added UF5: 74LS193, DIP-14_W7.62mm, F.Cu at (127.6, 208.5)
- added UF6: 74LS670, DIP-14_W7.62mm, F.Cu at (153.0, 208.5)
- added UF7: 74LS367, DIP-14_W7.62mm, F.Cu at (178.4, 208.5)
- added UF9: 74LS175, DIP-14_W7.62mm, F.Cu at (229.2, 208.5)
- added UH4: 74LS157, DIP-14_W7.62mm, F.Cu at (102.2, 170.4)
- added UH5: 74LS193, DIP-14_W7.62mm, F.Cu at (127.6, 170.4)
- added UH6: 74LS670, DIP-14_W7.62mm, F.Cu at (153.0, 170.4)
- added UH7: 74LS367, DIP-14_W7.62mm, F.Cu at (178.4, 170.4)
- added UJ1: 8316E, DIP-14_W7.62mm, F.Cu at (26.0, 151.3)
- added UJ10: 74S74, DIP-14_W7.62mm, F.Cu at (254.6, 151.3)
- added UJ6: 74LS191, DIP-14_W7.62mm, F.Cu at (153.0, 151.3)
- added UJ7: 74LS42, DIP-14_W7.62mm, F.Cu at (178.4, 151.3)
- added UJ8: 74LS175, DIP-14_W7.62mm, F.Cu at (203.8, 151.3)
- added UJ9: 74LS11, DIP-14_W7.62mm, F.Cu at (229.2, 151.3)
- added UK1: 8316E, DIP-14_W7.62mm, F.Cu at (26.0, 132.3)
- added UK10: 74LS32, DIP-14_W7.62mm, F.Cu at (254.6, 132.3)
- added UK6: 74LS161, DIP-14_W7.62mm, F.Cu at (153.0, 132.3)
- added UK7: 82S129, DIP-14_W7.62mm, F.Cu at (178.4, 132.3)
- added UK8: 74LS175, DIP-14_W7.62mm, F.Cu at (203.8, 132.3)
- added UK9: 74S02, DIP-14_W7.62mm, F.Cu at (229.2, 132.3)
- added UL1: 8316E, DIP-14_W7.62mm, F.Cu at (26.0, 113.2)
- added UL4: 74LS161, DIP-14_W7.62mm, F.Cu at (102.2, 113.2)
- added UL6: 74LS161, DIP-14_W7.62mm, F.Cu at (153.0, 113.2)
- added UL7: 74LS174, DIP-14_W7.62mm, F.Cu at (178.4, 113.2)
- added UL8: 74S260, DIP-14_W7.62mm, F.Cu at (203.8, 113.2)
- added UL9: 74LS74, DIP-14_W7.62mm, F.Cu at (229.2, 113.2)
- added UM5: 74LS20, DIP-14_W7.62mm, F.Cu at (127.6, 94.2)
- added UM6: 74LS161, DIP-14_W7.62mm, F.Cu at (153.0, 94.2)
- added UM8: 74LS32, DIP-14_W7.62mm, F.Cu at (203.8, 94.2)
- added UM9: 74LS74, DIP-14_W7.62mm, F.Cu at (229.2, 94.2)
- added UN1: 8316E, DIP-14_W7.62mm, F.Cu at (26.0, 75.2)
- added UN6: 74LS161, DIP-14_W7.62mm, F.Cu at (153.0, 75.2)
- added UN7: 74LS27, DIP-14_W7.62mm, F.Cu at (178.4, 75.2)
- added UN8: 74LS109, DIP-14_W7.62mm, F.Cu at (203.8, 75.2)
- added UN9: 74LS02, DIP-14_W7.62mm, F.Cu at (229.2, 75.2)
- added UP2: 74LS245, DIP-14_W7.62mm, F.Cu at (51.4, 56.1)

Commit message: Draw every device at its real package size
The board maps existed to answer "which chip is at C4", and then drew a
24-pin ROM and a 20-pin LS245 as the same 14-pin outline. package_for()
read pin counts from DEVICES, which holds 20 Pong-era parts against the
112 part types the boards actually use, and silently fell back to DIP-14
for the other 92.

tools/packages.py is the pin-count table, kept separate from devices.py
on purpose: packaging needs one number for every part on every board,
while devices.py carries verified pinouts for the parts validate_nets.py
reasons about, and widening that set to satisfy a drawing would let the
extractor trust readings nothing has checked.

688 of 704 devices now size. check_packages.py re-derives 56 of the
entries from KiCAD's symbol library — comparing the highest pin number,
not the pin count, since KiCAD omits no-connects and a 7493 symbol has
ten pins on a DIP-14 — and confirms all 20 parts in DEVICES agree. The
Am2901 slices and the POKEY come from DIP-40 stated on the Battlezone
sheet; the 8316E from the drawing's note that a 2708 may be fitted
instead.

What does not size is now said out loud rather than quietly drawn at 14
pins: four descriptions recorded where the sheet gave no part number,
and the Atari 0351xx ROM/PROM numbers, which get the class default and
are listed as unverified until someone has a board in front of them.

Two things found while reading the corpus for packages, both logged in
asteroids.read.json rather than acted on. The -06 rate multiplier
resolution was recorded and never applied to the board data, and the
parts list disagrees with both readings on designators. F4/H4/J4 take
either an LS670 or an LS170, and the 19-007 pull-up network is fitted
only with the LS170 — same package either way, but a real failure mode.

Also: republishing a board without --machine used to unlink it from its
machine, because most definitions carry no machine of their own and the
link lived only in boards.json. publish_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
Parts:
- UA1, UA2, UB1, UB2, UC1, UC2, UD1, UD2, UH2, UJ2: footprint DIP-14_W7.62mm -> DIP-18_W7.62mm
- UA3, UB3, UE1, UE3, UF1, UF3, UJ1, UK1, UL1, UN1: footprint DIP-14_W7.62mm -> DIP-24_W15.24mm
- UA5, UA6, UB4, UB5, UC4, UC5, UC9, UD4, UD5, UD6, UE4, UE5, UE6, UF10, UF4, UF5, UF6, UF7, UF9, UH4, UH5, UH6, UH7, UJ6, UJ7, UJ8, UK5, UK6, UK7, UK8, UL4, UL6, UL7, UM2, UM6, UN4, UN6, UN8: footprint DIP-14_W7.62mm -> DIP-16_W7.62mm
- UC8, UF2, UK3, UN11, UN2, UP11, UP2, UP4, UR11: footprint DIP-14_W7.62mm -> DIP-20_W7.62mm
- UL3: footprint DIP-14_W7.62mm -> DIP-40_W15.24mm

Commit message: Drop two grid rows that do not exist, and span the devices that do
Atari's grid alphabet skips G, I, O and Q, and the board definitions
listed G and Q as rows. Every device below F was therefore drawn a row
too low, the rendered board carried two empty bands, and F/H1 looked
like a three-position span for a part 1.2in long on a 0.75in pitch.

Confirmed three ways before touching it. Nothing in any read, signature
or signal record in this repo sits in a G or Q row, while both
neighbours of each are populated on the two densest boards — Battlezone
P:6 R:2, Asteroids-03 P:4 R:3. The sheets' own spanning designators
treat F and H as adjacent and H and J as adjacent, which is only
possible if G and I are not positions. And with G removed, F/H falls out
as an adjacent pair, which is what a 24-pin ROM needs. Pong predates the
convention and legitimately uses G, so it keeps its grid.

Spans are now data rather than prose. A device drawn across two or three
cells is still keyed at its first cell, because that is the only thing
`ics` may be keyed by, but the sheet's own designator goes in a `spans`
map and the footprint is placed at the mean of the cells it names. A
DIP-40 at B/C2 sits between B2 and C2 instead of hanging equally over A2
and C2. The build rejects a span whose rows are not adjacent — that
failure almost always means the grid is wrong, not the span.

Two more inconsistencies found and logged rather than guessed at. Two of
the Math Box's four Am2901 slices carry a span and two do not, though
all four are the same DIP-40 on the same pitch. And asteroids-04.json
carries five devices at the -03 PROM positions alongside the -04 ROMs
and is missing 035144-02 at D/E1, contradicting the substitution table,
memory_by_revision and its own status text in the same breath.

Co-Authored-By: Claude Opus 5 <noreply@anthropic.com>
Parts:
- moved UB3 47.6 mm to (76.8, 237.1)
- moved UF1 47.6 mm to (26.0, 160.9)
- moved UF3 47.6 mm to (76.8, 160.9)
- moved UA1 38.1 mm to (26.0, 265.6)
- moved UA2 38.1 mm to (51.4, 265.6)
- moved UA3 38.1 mm to (76.8, 265.6)
- moved UA5 38.1 mm to (127.6, 265.6)
- moved UA6 38.1 mm to (153.0, 265.6)
- moved UE1 38.1 mm to (26.0, 189.4)
- moved UE3 38.1 mm to (76.8, 189.4)
- moved UE4 38.1 mm to (102.2, 189.4)
- moved UE5 38.1 mm to (127.6, 189.4)
- moved UE6 38.1 mm to (153.0, 189.4)
- moved UB1 38.1 mm to (26.0, 246.6)
- moved UB2 38.1 mm to (51.4, 246.6)
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
Commit message: Name the four parts the sheets never did
C5, E12 and M12 on Asteroids were recorded by function — "counter",
"op-amp", "DIP switch" — because the drawings give no part number for
them, and they were the last devices the board maps could not size. The
parts lists give all three, and agree across printings.

C5 is a 9316. Five printings name a counter there: the 6th, 7th and
Cocktail 3rd say 37-9316, the 1st and 2nd say 37-74LS161, and the 9316
is Fairchild's 74161, so those are the same part and not a conflict. It
matches the read's own note that C5 divides 3kHz by 12 for the NMI.

E12 is Atari 137108-001, item 130, "Operational Amplifier Integrated
Circuit", at E12 in three printings; the Caberat manual names the type,
TL081CP. Same designator, same block, three documents. The same item
also lists a B/C12 location that nothing in the read accounts for, which
is noted and not acted on.

M12 is Atari 66-114P1T, a 4-station DIP switch, item 143 at M12 in three
printings. Sized as DIP-8, since n SPST switches in a DIP is 2n pins;
the 8-station switches on Battlezone and Tempest are DIP-16 for the same
reason.

All three are cross-document confirmations rather than re-readings of
the same sheet, which is the route the house rules say to try first and
the one that has resolved every conflict here so far. Every device on
every board now has a package: 106 of 106 part types, 694 of 694
devices. What remains unverified is the twenty Atari 0351xx ROM/PROM
positions, drawn on a class default, and those want a board.

Co-Authored-By: Claude Opus 5 <noreply@anthropic.com>
Parts:
- UM10, UP10: footprint DIP-14_W7.62mm -> DIP-16_W7.62mm

Commit message: Split multi-PCB manuals by figure, and take Battlezone through
A manual covering more than one PCB gives each its own parts-list figure,
and the heading names the board. Without using that, Battlezone's two
boards land in one heap and their designators collide — which AGENTS.md
already warns about in the drawings: C1 on one is not C1 on the other,
and both have a +5V LED called CR2. Rows now carry the figure they sit
under and --figure filters on it.

Battlezone is the result worth trusting the method on. It is the most
carefully hand-read board in the project, 97 devices off six sheet
sides, and across both PCBs the parts lists confirm 87 of 87 overlapping
designators with no disagreement at all. That says the harvest is sound
and that the six-sheet read was, and it recasts the 21 disagreements on
Asteroids as more likely errors in that read than noise in the lists.
The game PCB gains 8 devices and the Auxiliary 1 — small numbers, but
the confirmation is the point.

Also fixes a real loss this merge caused on its first run. The chip
lookup holds more than `ics` does: crystals, transistors, resistor
packs, a test point — everything on the board that is not on the
letter-number grid and so cannot be drawn. Rebuilding the lookup from
`ics` alone dropped twelve hand-read Battlezone devices and one on the
Auxiliary PCB. They are carried through now, and the hazard is written
into AGENTS.md next to the warning I had already put there and then
walked straight into.

Co-Authored-By: Claude Opus 5 <noreply@anthropic.com>
Parts:
- added UC7: 74LS174, DIP-16_W7.62mm, F.Cu at (178.4, 227.6)
- added UD7: 74LS86, DIP-14_W7.62mm, F.Cu at (178.4, 208.5)
- added UF8: 74LS175, DIP-16_W7.62mm, F.Cu at (203.8, 170.4)
- added UH10: 74LS74, DIP-14_W7.62mm, F.Cu at (254.6, 151.3)
- added UH11: 7404, DIP-14_W7.62mm, F.Cu at (280.0, 151.3)
- added UH8: 74LS399, DIP-16_W7.62mm, F.Cu at (203.8, 151.3)
- added UM11: 74LS174, DIP-16_W7.62mm, F.Cu at (280.0, 75.2)
- added UP9: 74LS164, DIP-14_W7.62mm, F.Cu at (229.2, 37.0)

Commit message: Put MAME's ROM positions on the maps; let the late Asteroids boards take the lists
Two things declined earlier as decisions rather than chores, reconsidered.

The parts-list harvest never reaches memory. Atari stocks ROMs and PROMs under
its own part numbers, not as 37-series IC stock, so those rows fail the
checksum the harvest depends on — which is why Red Baron's whole complement was
missing once, and why 79 memory cells on 15 boards sat empty with everything
around them filled. MAME has them: its ROM file names encode the board
position — 035224.e2 is part 035224 at E2, 037587-01.fh1 is at the span F/H1 —
and they were checked against real boards by the people who dumped them. The
site already publishes those maps as their own asset with their own caveat.
This is that source reaching the board map under the same label, not a new one
mixed in quietly: 78 devices on 14 boards, each recorded in the chip lookup as
"MAME ROM map", only where the map had nothing. The three cells where a parts
list and MAME disagree are untouched and stay logged.

Asteroids -05 and -06 were left without the parts lists because those are
written in early designators and a direct merge would put a device one column
from where the board has it. So they take -03's parts-list additions instead,
shifted through the drawing's early-to-late table where an alternate is known
and placed at the early cell otherwise — which is exactly what these boards
already do for their 78 unshifted drawing-read devices, under a caveat they
already carry. 13 each. None of the 22 turned out to have a known alternate,
and 9 land on cells a shifted device already occupies and are skipped rather
than duplicated. All of it runs inside the generator, so it survives
regeneration.

50 boards, 2,672 devices.

Co-Authored-By: Claude Fable 5.1 <noreply@anthropic.com>
Parts:
- added UH1: 036413-01, DIP-14_W7.62mm, F.Cu at (26.0, 151.3)
