File: kicad/lunar-lander/lunar-lander.kicad_pcb (KiCad board)
At the start: 2 copper layers, 300 x 300 mm, 6 parts

Commit message: Draw every device at its real package size
The board maps existed to answer "which chip is at C4", and then drew a
24-pin ROM and a 20-pin LS245 as the same 14-pin outline. package_for()
read pin counts from DEVICES, which holds 20 Pong-era parts against the
112 part types the boards actually use, and silently fell back to DIP-14
for the other 92.

tools/packages.py is the pin-count table, kept separate from devices.py
on purpose: packaging needs one number for every part on every board,
while devices.py carries verified pinouts for the parts validate_nets.py
reasons about, and widening that set to satisfy a drawing would let the
extractor trust readings nothing has checked.

688 of 704 devices now size. check_packages.py re-derives 56 of the
entries from KiCAD's symbol library — comparing the highest pin number,
not the pin count, since KiCAD omits no-connects and a 7493 symbol has
ten pins on a DIP-14 — and confirms all 20 parts in DEVICES agree. The
Am2901 slices and the POKEY come from DIP-40 stated on the Battlezone
sheet; the 8316E from the drawing's note that a 2708 may be fitted
instead.

What does not size is now said out loud rather than quietly drawn at 14
pins: four descriptions recorded where the sheet gave no part number,
and the Atari 0351xx ROM/PROM numbers, which get the class default and
are listed as unverified until someone has a board in front of them.

Two things found while reading the corpus for packages, both logged in
asteroids.read.json rather than acted on. The -06 rate multiplier
resolution was recorded and never applied to the board data, and the
parts list disagrees with both readings on designators. F4/H4/J4 take
either an LS670 or an LS170, and the 19-007 pull-up network is fitted
only with the LS170 — same package either way, but a real failure mode.

Also: republishing a board without --machine used to unlink it from its
machine, because most definitions carry no machine of their own and the
link lived only in boards.json. publish_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
Parts:
- UN5: footprint DIP-14_W7.62mm -> DIP-16_W7.62mm

Commit message: Drop two grid rows that do not exist, and span the devices that do
Atari's grid alphabet skips G, I, O and Q, and the board definitions
listed G and Q as rows. Every device below F was therefore drawn a row
too low, the rendered board carried two empty bands, and F/H1 looked
like a three-position span for a part 1.2in long on a 0.75in pitch.

Confirmed three ways before touching it. Nothing in any read, signature
or signal record in this repo sits in a G or Q row, while both
neighbours of each are populated on the two densest boards — Battlezone
P:6 R:2, Asteroids-03 P:4 R:3. The sheets' own spanning designators
treat F and H as adjacent and H and J as adjacent, which is only
possible if G and I are not positions. And with G removed, F/H falls out
as an adjacent pair, which is what a 24-pin ROM needs. Pong predates the
convention and legitimately uses G, so it keeps its grid.

Spans are now data rather than prose. A device drawn across two or three
cells is still keyed at its first cell, because that is the only thing
`ics` may be keyed by, but the sheet's own designator goes in a `spans`
map and the footprint is placed at the mean of the cells it names. A
DIP-40 at B/C2 sits between B2 and C2 instead of hanging equally over A2
and C2. The build rejects a span whose rows are not adjacent — that
failure almost always means the grid is wrong, not the span.

Two more inconsistencies found and logged rather than guessed at. Two of
the Math Box's four Am2901 slices carry a span and two do not, though
all four are the same DIP-40 on the same pitch. And asteroids-04.json
carries five devices at the -03 PROM positions alongside the -04 ROMs
and is missing 035144-02 at D/E1, contradicting the substitution table,
memory_by_revision and its own status text in the same breath.

Co-Authored-By: Claude Opus 5 <noreply@anthropic.com>
Parts:
- moved UN5 19.1 mm to (127.6, 56.1)
- moved UN6 19.1 mm to (153.0, 56.1)
- moved UM5 19.0 mm to (127.6, 75.2)
- moved UM6 19.0 mm to (153.0, 75.2)
- moved UM7 19.0 mm to (178.4, 75.2)

Commit message: Bring Missile Command and Lunar Lander through the same merge
Missile Command goes from 14 devices to 83, Lunar Lander from 6 to 60.
Both keep every device their drawing read already had, and every added
device records how many printings attest it.

Missile Command's five printings agree with each other on all 82
designators and confirm 12 of the 14 hand-read devices. The thirteenth,
D3, they dispute unanimously: all five call it a 74LS14 where the
drawing says 7404. The drawing keeps the cell, because the rule is that
a drawing read is someone looking at the board — but five against one is
worth knowing at the bench, so the dispute is now written into that
row's note and its source badge rather than buried in a log. The two
parts are both hex inverters on the same pinout, which is the pair a
drawing makes easiest to confuse.

Lunar Lander's three printings split on L6, E7 and E8 — some say
74LS170, others 74LS42, and a register file against a BCD decoder is not
a family misread, so one set is simply wrong and none of the three cells
is placed. Nine more designators appear in only one printing and are
left out; that manual's 1st printing carries 63 designators against the
3rd's 28, so those are mostly later printings not reprinting the list.

Two extraction fixes, both found by the packaging table refusing to size
what came out. Length was the wrong tie-break between two OCR readings
of a device name: '74S32' misread as '74832' is longer, and it parses as
a 74-series part with function number 832. What exposes it is that the
digits it actually ends in are 32, and 832 is not what follows a real
family — so the preference is now the spelling that decomposes as 74
plus a real family plus the device's own function number. That removed
74832, 74874 and 74L814 from three boards. The genuine parts the same
run surfaced — 7407, 74125, 74LS166, 74LS195, 74LS399 — join the
packaging table, verified against KiCAD, so all 901 devices still size.

Co-Authored-By: Claude Opus 5 <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
Parts:
- added UA10: 74LS399, DIP-16_W7.62mm, F.Cu at (254.6, 265.6)
- added UA7: 74LS74, DIP-14_W7.62mm, F.Cu at (178.4, 265.6)
- added UA9: 74LS109, DIP-16_W7.62mm, F.Cu at (229.2, 265.6)
- added UB10: 74LS399, DIP-16_W7.62mm, F.Cu at (254.6, 246.6)
- added UB2: 74LS244, DIP-20_W7.62mm, F.Cu at (51.4, 246.6)
- added UB4: 74LS393, DIP-14_W7.62mm, F.Cu at (102.2, 246.6)
- added UB7: 74LS191, DIP-16_W7.62mm, F.Cu at (178.4, 246.6)
- added UC10: 74LS399, DIP-16_W7.62mm, F.Cu at (254.6, 227.6)
- added UC2: 74LS244, DIP-20_W7.62mm, F.Cu at (51.4, 227.6)
- added UC7: 74LS191, DIP-16_W7.62mm, F.Cu at (178.4, 227.6)
- added UC9: 74LS191, DIP-16_W7.62mm, F.Cu at (229.2, 227.6)
- added UD10: 74LS399, DIP-16_W7.62mm, F.Cu at (254.6, 208.5)
- added UD4: 74LS74, DIP-14_W7.62mm, F.Cu at (102.2, 208.5)
- added UD5: 74LS393, DIP-14_W7.62mm, F.Cu at (127.6, 208.5)
- added UD7: 74LS191, DIP-16_W7.62mm, F.Cu at (178.4, 208.5)
- added UD8: 74LS174, DIP-16_W7.62mm, F.Cu at (203.8, 208.5)
- added UD9: 74LS191, DIP-16_W7.62mm, F.Cu at (229.2, 208.5)
- added UE10: 74LS399, DIP-16_W7.62mm, F.Cu at (254.6, 189.4)
- added UE3: 74LS245, DIP-20_W7.62mm, F.Cu at (76.8, 189.4)
- added UE4: 74LS139, DIP-16_W7.62mm, F.Cu at (102.2, 189.4)
- added UE9: 74LS191, DIP-16_W7.62mm, F.Cu at (229.2, 189.4)
- added UF10: 74LS399, DIP-16_W7.62mm, F.Cu at (254.6, 170.4)
- added UF3: 74LS157, DIP-16_W7.62mm, F.Cu at (76.8, 170.4)
- added UF4: 74LS670, DIP-16_W7.62mm, F.Cu at (102.2, 170.4)
- added UF5: 74LS191, DIP-16_W7.62mm, F.Cu at (127.6, 170.4)
- added UF6: 74LS157, DIP-16_W7.62mm, F.Cu at (153.0, 170.4)
- added UF7: 74LS273, DIP-20_W7.62mm, F.Cu at (178.4, 170.4)
- added UF8: 7497, DIP-16_W7.62mm, F.Cu at (203.8, 170.4)
- added UF9: 74LS191, DIP-16_W7.62mm, F.Cu at (229.2, 170.4)
- added UH3: 74LS157, DIP-16_W7.62mm, F.Cu at (76.8, 151.3)
- added UH4: 74LS670, DIP-16_W7.62mm, F.Cu at (102.2, 151.3)
- added UH6: 74LS367, DIP-16_W7.62mm, F.Cu at (153.0, 151.3)
- added UH7: 74LS273, DIP-20_W7.62mm, F.Cu at (178.4, 151.3)
- added UH8: 7497, DIP-16_W7.62mm, F.Cu at (203.8, 151.3)
- added UH9: 74LS191, DIP-16_W7.62mm, F.Cu at (229.2, 151.3)
- added UJ3: 74LS157, DIP-16_W7.62mm, F.Cu at (76.8, 132.3)
- added UJ4: 74LS670, DIP-16_W7.62mm, F.Cu at (102.2, 132.3)
- added UJ5: 74LS191, DIP-16_W7.62mm, F.Cu at (127.6, 132.3)
- added UJ6: 74LS367, DIP-16_W7.62mm, F.Cu at (153.0, 132.3)
- added UJ7: 74LS273, DIP-20_W7.62mm, F.Cu at (178.4, 132.3)
- added UJ8: 7497, DIP-16_W7.62mm, F.Cu at (203.8, 132.3)
- added UJ9: 74LS191, DIP-16_W7.62mm, F.Cu at (229.2, 132.3)
- added UK10: 74LS251, DIP-16_W7.62mm, F.Cu at (254.6, 113.2)
- added UK3: 74LS157, DIP-16_W7.62mm, F.Cu at (76.8, 113.2)
- added UK7: 74LS273, DIP-20_W7.62mm, F.Cu at (178.4, 113.2)
- added UK8: 7497, DIP-16_W7.62mm, F.Cu at (203.8, 113.2)
- added UL3: 74LS139, DIP-16_W7.62mm, F.Cu at (76.8, 94.2)
- added UM10: 74LS367, DIP-16_W7.62mm, F.Cu at (254.6, 75.2)
- added UN11: 74LS174, DIP-16_W7.62mm, F.Cu at (280.0, 56.1)
- added UN8: 74LS253, DIP-16_W7.62mm, F.Cu at (203.8, 56.1)
- added UN9: 74LS244, DIP-20_W7.62mm, F.Cu at (229.2, 56.1)
- added UP10: 74LS191, DIP-16_W7.62mm, F.Cu at (254.6, 37.0)
- added UP9: 74LS191, DIP-16_W7.62mm, F.Cu at (229.2, 37.0)
- added UR2: 74LS245, DIP-20_W7.62mm, F.Cu at (51.4, 18.0)

Commit message: Place the memory devices the IC parts lists cannot reach
Atari stocks ROM, RAM and the microprocessor under its own part numbers
— 90-7033, 036175-01, 90-6013 — not as 37-series IC stock, so the IC
harvest cannot see them however well it reads. That is why Centipede's
ROMs were missing and Red Baron's map had ten devices. merge_memory.py
reads those rows from the same typeset parts lists, under the same rules
as the IC merge: the drawing wins where it exists, two documents must
agree, and nothing is placed whose package cannot be established.

Red Baron 10 to 15, Asteroids Deluxe 92 to 100, Tempest 83 to 88,
Centipede 93 to 95, Missile Command 83 to 85, Lunar Lander 60 to 62.
1,494 devices across the boards, all sized, none contradicted.

Establishing the packages took two corrections, and both were the same
mistake in different clothes.

The first attempt sized Atari stock numbers by correlating a part
against the contact count of the socket at the positions it occupies,
pooled across a machine's documents. That is not a near miss: it put the
2114 at 40 pins, on twelve positions of apparent evidence, because two
printings number the board differently and the correlation was reading
one printing's parts list against another's sockets. Confined to within
a single document it behaves — 33 stock numbers established, 90-6013 by
39 documents agreeing, and 90-7033 correctly refusing to answer rather
than answering wrongly. Those 33 are in packages.py with their
provenance.

The second was the same shape. MAME's dump size was sizing a part from
whatever MAME dumped at that cell, which on Red Baron meant sizing
036175-01 from a dump of 037000-01 — sizing the socket, not the chip.
MAME now sizes a part only when the dump is of that part. Red Baron
loses two devices and keeps thirteen that are right.

Four more parts are sized from MAME's dump sizes alone, where every set
carrying the part agrees and the era leaves no room: 32 bytes and 256
bytes are both bipolar PROMs in a 1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
Parts:
- added UC3: 90-6013, DIP-40_W15.24mm, F.Cu at (76.8, 227.6)
- added UC8: 034602-01, DIP-16_W7.62mm, F.Cu at (203.8, 227.6)

Commit message: Put MAME's ROM positions on the maps; let the late Asteroids boards take the lists
Two things declined earlier as decisions rather than chores, reconsidered.

The parts-list harvest never reaches memory. Atari stocks ROMs and PROMs under
its own part numbers, not as 37-series IC stock, so those rows fail the
checksum the harvest depends on — which is why Red Baron's whole complement was
missing once, and why 79 memory cells on 15 boards sat empty with everything
around them filled. MAME has them: its ROM file names encode the board
position — 035224.e2 is part 035224 at E2, 037587-01.fh1 is at the span F/H1 —
and they were checked against real boards by the people who dumped them. The
site already publishes those maps as their own asset with their own caveat.
This is that source reaching the board map under the same label, not a new one
mixed in quietly: 78 devices on 14 boards, each recorded in the chip lookup as
"MAME ROM map", only where the map had nothing. The three cells where a parts
list and MAME disagree are untouched and stay logged.

Asteroids -05 and -06 were left without the parts lists because those are
written in early designators and a direct merge would put a device one column
from where the board has it. So they take -03's parts-list additions instead,
shifted through the drawing's early-to-late table where an alternate is known
and placed at the early cell otherwise — which is exactly what these boards
already do for their 78 unshifted drawing-read devices, under a caveat they
already carry. 13 each. None of the 22 turned out to have a known alternate,
and 9 land on cells a shifted device already occupies and are skipped rather
than duplicated. All of it runs inside the generator, so it survives
regeneration.

50 boards, 2,672 devices.

Co-Authored-By: Claude Fable 5.1 <noreply@anthropic.com>
Parts:
- added UC1: 034570-01, DIP-14_W7.62mm, F.Cu at (26.0, 227.6)
- added UD1: 034571-02, DIP-14_W7.62mm, F.Cu at (26.0, 199.0)
- added UF1: 034572-02, DIP-14_W7.62mm, F.Cu at (26.0, 170.4)
- added UM3: 034597-01, DIP-14_W7.62mm, F.Cu at (76.8, 75.2)
- added UN3: 034598-01, DIP-14_W7.62mm, F.Cu at (76.8, 46.6)
- added UR3: 034599-01, DIP-14_W7.62mm, F.Cu at (76.8, 18.0)
