File: kicad/monte-carlo/monte-carlo.kicad_pcb (KiCad board)
At the start: 2 copper layers, 300 x 304.7 mm, 79 parts

Commit message: Drop a cell both readings claim, instead of taking the last one
locations() detects a designator claimed twice by the same parts list and
returns the collision alongside the mapping. harvest() took only
locations(...)[0] and dropped that half of the answer on the floor, so a
contested cell was resolved by whichever reading came last in the file.

22 devices on the published site were chosen that way: Food Fight 1, I-Robot 8,
Indy 4 3, Monte Carlo 4, Pole Position 6. They are withdrawn. merge only ever
adds cells, so re-running it could not undo them — they had to come off
explicitly. Both readings are recorded in each board's read file rather than
just deleted, because a repairer at the bench is better served by "it is one of
these two" than by a silent gap.

A contested cell is now kept only when every reading of it names the same
device — '74L886' against '74LS86' is one part and an OCR of S as 8, and Orbit's
three such cells stay. Anything else is dropped and printed.

It deliberately does NOT use plausible() to break the tie, though the
cross-printing split does. plausible() does not recognise the Fairchild 93xx and
96xx series: it calls 9312, 9322 and 9602 implausible, and 9316 too — which this
repo's own equivalence table documents as Fairchild's 74161. Filtering on it here
would have discarded the 9312 reading of Indy 4's B3 and "resolved" that cell to
a 7474, a different device entirely. A false correction is worse than the
collision it replaces. The split path has the same blind spot and is now flagged
in HANDOFF, unaudited.

The fix also unblocks the two boards withheld last time for exactly this reason.
Pole Position II (38 devices, 8 cells dropped) and Xevious (18, 1 dropped) no
longer need figure-splitting to be safe, because a cell nothing can attribute is
now simply absent rather than guessed.

47 boards, 2,489 devices.

Co-Authored-By: Claude Opus 5 <noreply@anthropic.com>
Parts:
- removed UA6, UH8, UP7: 74LS374, DIP-20_W7.62mm
- removed UB1: 74LS241, DIP-20_W7.62mm

Commit message: Teach plausible() the Fairchild parts; audit what it had decided
The last commit flagged that plausible() does not recognise the Fairchild
93xx/96xx series and left it unaudited. Audited now.

plausible() called 9312, 9316, 9321, 9322, 9300, 9301, 9334 and 9602
implausible — eight parts in 111 trusted rows and on 64 devices of published
maps, every one of them admitted by well_formed(). The two functions disagreed
about real parts, and 9316 is one this repo's own equivalence table documents
as Fairchild's 74161. Bounded to 9[36]\d{2}: a bare 9\d{3} would admit any
four-digit OCR smear.

The audit replayed the cross-printing split over every published board. 8 cells
had been decided by the filter. 4 were Asteroids P9, where a printing reading
9316 lost to one reading 74LS164 — the blind spot, discarding the more specific
reading as wreckage — and P9 is on none of the four Asteroids maps. The other 4
were the filter doing its job: 8728 to 8T28 on Football, 74LSI91 to 74LS191 on
Major Havoc, capital-I read as 1. After the fix 4 remain, all of the second
kind. No published device ever came from a false resolution.

Dropping a contested cell frees the readings a collision used to consume, so a
re-merge recovers 9 devices: Monte Carlo 3, Pole Position 4, Food Fight 1,
Soccer 1. Checked first that none of the 22 cells withdrawn last commit would
come back — every one is still reported as contested.

APB exposed a separate fault. Its 3B/F span names rows five apart, build_board
raised on it, and removing it by hand did not stick because the next merge wrote
it again — the adjacency rule lived only at build time, after the board file was
already wrong. It now runs where the designator is first accepted, and says so:
"impossible span 3B/F — those rows are not adjacent on this grid".

All 47 boards build. 2,498 devices.

Co-Authored-By: Claude Opus 5 <noreply@anthropic.com>
Parts:
- added UE2: 74LS245, DIP-20_W7.62mm, F.Cu at (51.4, 189.4)
- added UJ6: 74LS245, DIP-20_W7.62mm, F.Cu at (153.0, 132.3)
- added UK4: 74LS245, DIP-20_W7.62mm, F.Cu at (102.2, 113.2)

Commit message: Put MAME's ROM positions on the maps; let the late Asteroids boards take the lists
Two things declined earlier as decisions rather than chores, reconsidered.

The parts-list harvest never reaches memory. Atari stocks ROMs and PROMs under
its own part numbers, not as 37-series IC stock, so those rows fail the
checksum the harvest depends on — which is why Red Baron's whole complement was
missing once, and why 79 memory cells on 15 boards sat empty with everything
around them filled. MAME has them: its ROM file names encode the board
position — 035224.e2 is part 035224 at E2, 037587-01.fh1 is at the span F/H1 —
and they were checked against real boards by the people who dumped them. The
site already publishes those maps as their own asset with their own caveat.
This is that source reaching the board map under the same label, not a new one
mixed in quietly: 78 devices on 14 boards, each recorded in the chip lookup as
"MAME ROM map", only where the map had nothing. The three cells where a parts
list and MAME disagree are untouched and stay logged.

Asteroids -05 and -06 were left without the parts lists because those are
written in early designators and a direct merge would put a device one column
from where the board has it. So they take -03's parts-list additions instead,
shifted through the drawing's early-to-late table where an alternate is known
and placed at the early cell otherwise — which is exactly what these boards
already do for their 78 unshifted drawing-read devices, under a caveat they
already carry. 13 each. None of the 22 turned out to have a known alternate,
and 9 land on cells a shifted device already occupies and are skipped rather
than duplicated. All of it runs inside the generator, so it survives
regeneration.

50 boards, 2,672 devices.

Co-Authored-By: Claude Fable 5.1 <noreply@anthropic.com>
Parts:
- added UC1: 35763-01, DIP-14_W7.62mm, F.Cu at (26.0, 227.6)
- added UE6: 35775-01, DIP-14_W7.62mm, F.Cu at (153.0, 189.4)
- added UE7: 35785-01, DIP-14_W7.62mm, F.Cu at (178.4, 189.4)
- added UF1: 35765-01, DIP-14_W7.62mm, F.Cu at (26.0, 170.4)
- added UH1: 35766-01, DIP-14_W7.62mm, F.Cu at (26.0, 151.3)
- added UM4: 35778-01, DIP-14_W7.62mm, F.Cu at (102.2, 75.2)
- added UM6: 35779-01, DIP-14_W7.62mm, F.Cu at (153.0, 75.2)
