File: kicad/orbit/orbit.kicad_pcb (KiCad board)
At the start: 2 copper layers, 350.8 x 304.7 mm, 37 parts

Commit message: Put MAME's ROM positions on the maps; let the late Asteroids boards take the lists
Two things declined earlier as decisions rather than chores, reconsidered.

The parts-list harvest never reaches memory. Atari stocks ROMs and PROMs under
its own part numbers, not as 37-series IC stock, so those rows fail the
checksum the harvest depends on — which is why Red Baron's whole complement was
missing once, and why 79 memory cells on 15 boards sat empty with everything
around them filled. MAME has them: its ROM file names encode the board
position — 035224.e2 is part 035224 at E2, 037587-01.fh1 is at the span F/H1 —
and they were checked against real boards by the people who dumped them. The
site already publishes those maps as their own asset with their own caveat.
This is that source reaching the board map under the same label, not a new one
mixed in quietly: 78 devices on 14 boards, each recorded in the chip lookup as
"MAME ROM map", only where the map had nothing. The three cells where a parts
list and MAME disagree are untouched and stay logged.

Asteroids -05 and -06 were left without the parts lists because those are
written in early designators and a direct merge would put a device one column
from where the board has it. So they take -03's parts-list additions instead,
shifted through the drawing's early-to-late table where an alternate is known
and placed at the early cell otherwise — which is exactly what these boards
already do for their 78 unshifted drawing-read devices, under a caveat they
already carry. 13 each. None of the 22 turned out to have a known alternate,
and 9 land on cells a shifted device already occupies and are skipped rather
than duplicated. All of it runs inside the generator, so it survives
regeneration.

50 boards, 2,672 devices.

Co-Authored-By: Claude Fable 5.1 <noreply@anthropic.com>
Parts:
- added UL1: 033694, DIP-14_W7.62mm, F.Cu at (26.0, 94.2)
- added UL2: 033693, DIP-14_W7.62mm, F.Cu at (51.4, 94.2)
- added UM1: 033692, DIP-14_W7.62mm, F.Cu at (26.0, 75.2)
- added UM2: 033691, DIP-14_W7.62mm, F.Cu at (51.4, 75.2)
- added UN1: 033690, DIP-14_W7.62mm, F.Cu at (26.0, 56.1)
- added UN2: 033689, DIP-14_W7.62mm, F.Cu at (51.4, 56.1)
