File: kicad/tempest/tempest.kicad_pcb (KiCad board)
At the start: 2 copper layers, 300 x 300 mm, 93 parts

Commit message: Split two maps that were two PCBs stacked
The collision work catches a manual whose PCBs share designators: C1 on one is
not C1 on the other, the cell is claimed twice, something notices. It cannot
catch the quieter case. Two PCBs whose designators do not overlap merge into a
single map with no collision, no warning, and a result that looks complete.

Asking of every published board whether its trusted rows sat under more than one
figure heading naming a different PCB found two: I, Robot (an I, ROBOT CPU PCB
and an I, ROBOT Video PCB) and Paperboy (a Central Processing Unit PCB and a
Video PCB). Both published one map covering both boards. That is worse than an
incomplete map — a repairer reading cell 5A off it is being told something
false, because 5A exists on both boards and means different things.

Split. The existing slug keeps the CPU board, so its URL and anything pointing
at it stay valid, and the video board is new. Splitting recovers devices rather
than losing them — I, Robot goes from 45 to 33 plus 24 — because cells both
boards claimed had been dropped as collisions and are separable once the boards
are.

Three more took a handful of devices from the wrong board's figure: Tempest 5
from its Auxiliary PCB on a map that is the Analog Vector-Generator PCB, Pole
Position 4 sitting under a video-display monitor list as readily as the CPU one,
Food Fight 1 shared with an EMI Shield figure. Removed and re-harvested under
each board's own figure, where all three add nothing back — which is what
confirms the five, four and one were never theirs.

Millipede looked identical and is not. Its TM-217 has one figure heading the
regex recognises, so all 46 rows inherit 'Utility Panel Assembly' — but they are
game-PCB TTL and a utility panel does not carry 46 logic chips. Meaningless
attribution rather than a wrong board, and its two printings agree. Left alone.

Splitting also exposed that merge_ic_locations keeps lookup entries not on the
grid, by design, for crystals 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
Parts:
- removed UA2: 74109, DIP-16_W7.62mm
- removed UA3, UH4: 74LS174, DIP-16_W7.62mm
- removed UJ3: 74LS175, DIP-16_W7.62mm
- removed UJ4: 74LS02, DIP-14_W7.62mm

Commit message: Put MAME's ROM positions on the maps; let the late Asteroids boards take the lists
Two things declined earlier as decisions rather than chores, reconsidered.

The parts-list harvest never reaches memory. Atari stocks ROMs and PROMs under
its own part numbers, not as 37-series IC stock, so those rows fail the
checksum the harvest depends on — which is why Red Baron's whole complement was
missing once, and why 79 memory cells on 15 boards sat empty with everything
around them filled. MAME has them: its ROM file names encode the board
position — 035224.e2 is part 035224 at E2, 037587-01.fh1 is at the span F/H1 —
and they were checked against real boards by the people who dumped them. The
site already publishes those maps as their own asset with their own caveat.
This is that source reaching the board map under the same label, not a new one
mixed in quietly: 78 devices on 14 boards, each recorded in the chip lookup as
"MAME ROM map", only where the map had nothing. The three cells where a parts
list and MAME disagree are untouched and stay logged.

Asteroids -05 and -06 were left without the parts lists because those are
written in early designators and a direct merge would put a device one column
from where the board has it. So they take -03's parts-list additions instead,
shifted through the drawing's early-to-late table where an alternate is known
and placed at the early cell otherwise — which is exactly what these boards
already do for their 78 unshifted drawing-read devices, under a caveat they
already carry. 13 each. None of the 22 turned out to have a known alternate,
and 9 land on cells a shifted device already occupies and are skipped rather
than duplicated. All of it runs inside the generator, so it survives
regeneration.

50 boards, 2,672 devices.

Co-Authored-By: Claude Fable 5.1 <noreply@anthropic.com>
Parts:
- added UF1: 136002-134, DIP-14_W7.62mm, F.Cu at (26.0, 170.4)
- added UJ1: 136002-235, DIP-14_W7.62mm, F.Cu at (26.0, 132.3)
- added UL1: 136002-136, DIP-14_W7.62mm, F.Cu at (26.0, 84.7)
