File: kicad/food-fight/food-fight.kicad_pcb (KiCad board)
At the start: 2 copper layers, 315 x 257 mm, 27 parts, among them U10C 7406, U10M 74LS161, U10N 74LS161, U1F 74LS86, U1H 7407, U2C 74S08, U2D 74S157, U2H 74LS74, U2K 74LS74, U3B 74LS157, U3P 74LS157, U4C 74LS86, U4F 74LS273, U4K 74LS367, U4L 74LS157, U4M 74LS157, U4N 74LS157, U4P 74S00, U5M 74LS194, U5N 74LS194, U6B 74LS273, U6H 74LS157, U6K 74LS273, U7M 74LS273, U8H 74LS245, U8M 74LS244, U8N 74LS244

Commit message: Read MAME's column-first maps; apply them only where the map is the same PCB
1,009 of MAME's 1,469 ROM maps are number-letter and ten transposed boards
have one, so the tool reads that convention now — 5JK is column 5, rows J/K —
and refuses a map whose style contradicts the board's: Millipede's and
Paperboy's boards are column-first with letter-first MAME maps, and reading one
convention as the other transposes a map without saying so.

Tested before applying anything: where a MAME ROM cell lands on a map, is the
device already there memory or logic? On Pole Position, twelve occupied cells
and twelve of them logic — 74LS74, 74LS139, 74LS373 — across seven printings
that agree with each other. Twelve for twelve is not OCR; it is another board's
grid. Pole Position is Namco CPU-plus-video hardware and the map is the CPU
board alone. Pole Position II is nine for nine the same. 720 Degrees and APB
share an identical 2B = 74LS153 against a ROM, and 9 and 13 positions on rows
the map does not have. Road Blasters puts 24 of 34 off the grid. Xevious's
off-grid ROMs are tagged pals_vidbd and sub-CPU program by MAME itself. Those
six take nothing, and each read file says why.

The four with zero conflicts and nothing off-grid that points to another board
take their positions: Return of the Jedi 13, Food Fight 12, Quantum 9, Super
Sprint 20. Every one labelled "MAME ROM map" in the chip lookup.

50 boards, 2,726 devices.

Co-Authored-By: Claude Fable 5.1 <noreply@anthropic.com>
Parts:
- added U2P: 136020-112, DIP-14_W7.62mm, F.Cu at (51.4, 18.0)
- added U4D: 136020-111, DIP-14_W7.62mm, F.Cu at (102.2, 170.4)
- added U4E: 136020-110, DIP-14_W7.62mm, F.Cu at (102.2, 151.3)
- added U6L: 136020-109, DIP-14_W7.62mm, F.Cu at (153.0, 65.6)
- added U8C: 136020-301, DIP-14_W7.62mm, F.Cu at (203.8, 189.4)
- added U8D: 136020-303, DIP-14_W7.62mm, F.Cu at (203.8, 170.4)
- added U8E: 136020-305, DIP-14_W7.62mm, F.Cu at (203.8, 151.3)
- added U8F: 136020-307, DIP-14_W7.62mm, F.Cu at (203.8, 132.3)
- added U9C: 136020-302, DIP-14_W7.62mm, F.Cu at (229.2, 189.4)
- added U9D: 136020-204, DIP-14_W7.62mm, F.Cu at (229.2, 170.4)
- added U9E: 136020-306, DIP-14_W7.62mm, F.Cu at (229.2, 151.3)
- added U9F: 136020-208, DIP-14_W7.62mm, F.Cu at (229.2, 132.3)
