File: kicad/quantum/quantum.kicad_pcb (KiCad board)
At the start: 2 copper layers, 290 x 257 mm, 49 parts, among them U10J 74LS04, U10K 74LS86, U10P 74LS157, U10R 74LS74, U1E 74LS244, U1F 74LS244, U1N 74LS245, U1P 74LS245, U2R 74LS74, U3P 74LS245, U4D 74LS245, U4E 74LS245, U4K 74LS08, U4M 7406, U4N 74S32, U4P 74LS00, U4R 74LS393, U5C 74LS157, U5H 74LS174, U5K 74LS27, U5L 74LS161, U5M 74LS161, U5N 74LS273, U5P 74LS74, U5R 74LS393, U6J 74LS42, U6K 74LS109, U6L 74LS14, U6M 74LS161, U6N 74S02, U6P 74S02, U7C 74LS194, U7D 74LS175, U7E 74LS157, U7H 74LS00, U7K 74LS32, U7L 74S260, U7M 74LS161, U8C 74LS194, U8D 74LS273, U8F 74LS175, U8K 74LS32, U8L 74S02, U8M 74LS191, U8N 74LS191, U8P 74S04, U9M 74LS244, U9N 74LS244, U9P 74LS191

Commit message: Read MAME's column-first maps; apply them only where the map is the same PCB
1,009 of MAME's 1,469 ROM maps are number-letter and ten transposed boards
have one, so the tool reads that convention now — 5JK is column 5, rows J/K —
and refuses a map whose style contradicts the board's: Millipede's and
Paperboy's boards are column-first with letter-first MAME maps, and reading one
convention as the other transposes a map without saying so.

Tested before applying anything: where a MAME ROM cell lands on a map, is the
device already there memory or logic? On Pole Position, twelve occupied cells
and twelve of them logic — 74LS74, 74LS139, 74LS373 — across seven printings
that agree with each other. Twelve for twelve is not OCR; it is another board's
grid. Pole Position is Namco CPU-plus-video hardware and the map is the CPU
board alone. Pole Position II is nine for nine the same. 720 Degrees and APB
share an identical 2B = 74LS153 against a ROM, and 9 and 13 positions on rows
the map does not have. Road Blasters puts 24 of 34 off the grid. Xevious's
off-grid ROMs are tagged pals_vidbd and sub-CPU program by MAME itself. Those
six take nothing, and each read file says why.

The four with zero conflicts and nothing off-grid that points to another board
take their positions: Return of the Jedi 13, Food Fight 12, Quantum 9, Super
Sprint 20. Every one labelled "MAME ROM map" in the chip lookup.

50 boards, 2,726 devices.

Co-Authored-By: Claude Fable 5.1 <noreply@anthropic.com>
Parts:
- added U2E: 136016-201, DIP-14_W7.62mm, F.Cu at (51.4, 189.4)
- added U2F: 136016-102, DIP-14_W7.62mm, F.Cu at (51.4, 170.4)
- added U2H: 136016-203, DIP-14_W7.62mm, F.Cu at (51.4, 141.8)
- added U2L: 136016-105, DIP-14_W7.62mm, F.Cu at (51.4, 94.2)
- added U3E: 136016-206, DIP-14_W7.62mm, F.Cu at (76.8, 189.4)
- added U3F: 136016-107, DIP-14_W7.62mm, F.Cu at (76.8, 170.4)
- added U3H: 136016-208, DIP-14_W7.62mm, F.Cu at (76.8, 141.8)
- added U3L: 136016-110, DIP-14_W7.62mm, F.Cu at (76.8, 94.2)
- added U6H: 136002-125, DIP-16_W7.62mm, F.Cu at (153.0, 151.3)
