File: kicad/return-of-the-jedi/return-of-the-jedi.kicad_pcb (KiCad board)
At the start: 2 copper layers, 392 x 314 mm, 37 parts, among them U10K 74LS74, U10L 74LS08, U10M 74S32, U11M 74LS20, U12E 74LS08, U12H 74LS00, U12N 74S32, U13H 74LS90, U13M 74S32, U14B 74LS257, U14J 74LS259, U1N 74LS00, U2A 74LS139, U2F 74LS273, U2H 74LS194, U2J 74LS194, U2N 74LS32, U2P 74LS245, U3A 74LS163A, U3H 74LS175, U3P 74LS32, U3T 74LS157, U4A 74LS30, U4D 74LS273, U4E 74LS374, U4F 74S08, U5B 74S02, U5C 74LS174, U5E 74LS374, U5M 74LS163A, U5R 74LS257, U6L 74LS245, U7K 74LS00, U8C 74S74, U8F 74LS86, U8M 74LS157, U8N 74LS157

Commit message: Read MAME's column-first maps; apply them only where the map is the same PCB
1,009 of MAME's 1,469 ROM maps are number-letter and ten transposed boards
have one, so the tool reads that convention now — 5JK is column 5, rows J/K —
and refuses a map whose style contradicts the board's: Millipede's and
Paperboy's boards are column-first with letter-first MAME maps, and reading one
convention as the other transposes a map without saying so.

Tested before applying anything: where a MAME ROM cell lands on a map, is the
device already there memory or logic? On Pole Position, twelve occupied cells
and twelve of them logic — 74LS74, 74LS139, 74LS373 — across seven printings
that agree with each other. Twelve for twelve is not OCR; it is another board's
grid. Pole Position is Namco CPU-plus-video hardware and the map is the CPU
board alone. Pole Position II is nine for nine the same. 720 Degrees and APB
share an identical 2B = 74LS153 against a ROM, and 9 and 13 positions on rows
the map does not have. Road Blasters puts 24 of 34 off the grid. Xevious's
off-grid ROMs are tagged pals_vidbd and sub-CPU program by MAME itself. Those
six take nothing, and each read file says why.

The four with zero conflicts and nothing off-grid that points to another board
take their positions: Return of the Jedi 13, Food Fight 12, Quantum 9, Super
Sprint 20. Every one labelled "MAME ROM map" in the chip lookup.

50 boards, 2,726 devices.

Co-Authored-By: Claude Fable 5.1 <noreply@anthropic.com>
Parts:
- added U01C: 136030-133, DIP-14_W7.62mm, F.Cu at (26.0, 246.6)
- added U01F: 136030-131, DIP-14_W7.62mm, F.Cu at (26.0, 189.4)
- added U01H: 136030-130, DIP-14_W7.62mm, F.Cu at (26.0, 170.4)
- added U01K: 136030-129, DIP-14_W7.62mm, F.Cu at (26.0, 132.3)
- added U01M: 136030-128, DIP-14_W7.62mm, F.Cu at (26.0, 94.2)
- added U06N: 136030-127, DIP-14_W7.62mm, F.Cu at (153.0, 75.2)
- added U06R: 136030-126, DIP-14_W7.62mm, F.Cu at (153.0, 37.0)
- added U11T: 136030-215, DIP-14_W7.62mm, F.Cu at (280.0, 18.0)
- added U13A: 136030-122, DIP-14_W7.62mm, F.Cu at (330.8, 284.7)
- added U13B: 136030-124, DIP-14_W7.62mm, F.Cu at (330.8, 265.6)
- added U13D: 136030-123, DIP-14_W7.62mm, F.Cu at (330.8, 227.6)
- added U13F: 136030-222, DIP-14_W7.62mm, F.Cu at (330.8, 189.4)
- added U14F: 136030-221, DIP-14_W7.62mm, F.Cu at (356.2, 189.4)
