File: kicad/super-sprint/super-sprint.kicad_pcb (KiCad board)
At the start: 2 copper layers, 315 x 295 mm, 31 parts, among them U10B 74S00, U10H 74LS244, U11C 74S00, U1A 74LS157, U1B 74LS157, U1D 74LS244, U1E 74LS244, U1K 74LS32, U1M 74LS245, U1S 74LS244, U1T 74S74, U2F 74LS139, U2H 74LS244, U2K 74LS174, U2L 74S74, U2M 74LS139, U2N 74LS374, U2R 74LS374, U2T 74S32, U3F 74LS153, U3H 74LS153, U3L 74LS153, U3M 74LS153, U4F 74LS273, U4K 74S74, U4M 74LS273, U5B 74LS109, U5K 74LS04, U5S 74LS273, U7E 74LS32, U8E 74LS163A

Commit message: Read MAME's column-first maps; apply them only where the map is the same PCB
1,009 of MAME's 1,469 ROM maps are number-letter and ten transposed boards
have one, so the tool reads that convention now — 5JK is column 5, rows J/K —
and refuses a map whose style contradicts the board's: Millipede's and
Paperboy's boards are column-first with letter-first MAME maps, and reading one
convention as the other transposes a map without saying so.

Tested before applying anything: where a MAME ROM cell lands on a map, is the
device already there memory or logic? On Pole Position, twelve occupied cells
and twelve of them logic — 74LS74, 74LS139, 74LS373 — across seven printings
that agree with each other. Twelve for twelve is not OCR; it is another board's
grid. Pole Position is Namco CPU-plus-video hardware and the map is the CPU
board alone. Pole Position II is nine for nine the same. 720 Degrees and APB
share an identical 2B = 74LS153 against a ROM, and 9 and 13 positions on rows
the map does not have. Road Blasters puts 24 of 34 off the grid. Xevious's
off-grid ROMs are tagged pals_vidbd and sub-CPU program by MAME itself. Those
six take nothing, and each read file says why.

The four with zero conflicts and nothing off-grid that points to another board
take their positions: Return of the Jedi 13, Food Fight 12, Quantum 9, Super
Sprint 20. Every one labelled "MAME ROM map" in the chip lookup.

50 boards, 2,726 devices.

Co-Authored-By: Claude Fable 5.1 <noreply@anthropic.com>
Parts:
- added U2B: 136042-419, DIP-14_W7.62mm, F.Cu at (51.4, 237.1)
- added U2D: 136042-420, DIP-14_W7.62mm, F.Cu at (51.4, 208.5)
- added U6A: 136042-105, DIP-14_W7.62mm, F.Cu at (153.0, 265.6)
- added U6B: 136042-106, DIP-14_W7.62mm, F.Cu at (153.0, 246.6)
- added U6C: 136042-107, DIP-14_W7.62mm, F.Cu at (153.0, 227.6)
- added U6D: 136042-108, DIP-14_W7.62mm, F.Cu at (153.0, 199.0)
- added U6F: 136042-109, DIP-14_W7.62mm, F.Cu at (153.0, 160.9)
- added U6K: 136042-127, DIP-14_W7.62mm, F.Cu at (153.0, 132.3)
- added U6L: 136042-126, DIP-14_W7.62mm, F.Cu at (153.0, 113.2)
- added U6M: 136042-114, DIP-14_W7.62mm, F.Cu at (153.0, 94.2)
- added U6N: 136042-325, DIP-14_W7.62mm, F.Cu at (153.0, 75.2)
- added U6R: 136042-117, DIP-14_W7.62mm, F.Cu at (153.0, 46.6)
- added U6S: 136042-122, DIP-14_W7.62mm, F.Cu at (153.0, 37.0)
- added U6T: 136042-118, DIP-14_W7.62mm, F.Cu at (153.0, 18.0)
- added U7A: 136042-101, DIP-14_W7.62mm, F.Cu at (178.4, 265.6)
- added U7B: 136042-102, DIP-14_W7.62mm, F.Cu at (178.4, 246.6)
- added U7C: 136042-103, DIP-14_W7.62mm, F.Cu at (178.4, 227.6)
- added U7D: 136042-104, DIP-14_W7.62mm, F.Cu at (178.4, 199.0)
- added U7L: 136042-330, DIP-14_W7.62mm, F.Cu at (178.4, 113.2)
- added U7N: 136042-331, DIP-14_W7.62mm, F.Cu at (178.4, 75.2)
